Commit message: Fix pre-commit linting, advice and suggestions

File: car_description/urdf/cameras.xacro (robot description, xacro)
@@ -3,5 +3,5 @@
   <xacro:macro name="camera_mount" params="name parent *origin">
     <joint name="${name}_joint" type="fixed">
-      <xacro:insert_block name="origin" />
+      <xacro:insert_block name="origin"/>
       <parent link="${parent}"/>
       <child link="${name}"/>
@@ -9,7 +9,7 @@
     <link name="${name}">
       <inertial>
-        <mass value="1e-5" />
+        <mass value="1e-5"/>
         <origin xyz="0 0 0" rpy="0 0 0"/>
-        <inertia ixx="1e-6" ixy="0" ixz="0" iyy="1e-6" iyz="0" izz="1e-6" />
+        <inertia ixx="1e-6" ixy="0" ixz="0" iyy="1e-6" iyz="0" izz="1e-6"/>
       </inertial>
     </link>

File: car_description/urdf/gps.xacro (robot description, xacro)
@@ -3,5 +3,5 @@
   <xacro:macro name="gps" params="name *origin">
     <joint name="${name}_joint" type="fixed">
-      <xacro:insert_block name="origin" />
+      <xacro:insert_block name="origin"/>
       <parent link="${roof_datum}"/>
       <child link="${name}"/>
@@ -9,7 +9,7 @@
     <link name="${name}">
       <inertial>
-        <mass value="1e-5" />
+        <mass value="1e-5"/>
         <origin xyz="0 0 0" rpy="0 0 0"/>
-        <inertia ixx="1e-6" ixy="0" ixz="0" iyy="1e-6" iyz="0" izz="1e-6" />
+        <inertia ixx="1e-6" ixy="0" ixz="0" iyy="1e-6" iyz="0" izz="1e-6"/>
       </inertial>
     </link>

File: car_description/urdf/imu.xacro (robot description, xacro)
@@ -3,5 +3,5 @@
   <xacro:macro name="imu" params="imu *origin">
     <joint name="${imu}_joint" type="fixed">
-      <xacro:insert_block name="origin" />
+      <xacro:insert_block name="origin"/>
       <parent link="${roof_datum}"/>
       <child link="${imu}"/>
@@ -9,7 +9,7 @@
     <link name="${imu}">
       <inertial>
-        <mass value="1e-5" />
+        <mass value="1e-5"/>
         <origin xyz="0 0 0" rpy="0 0 0"/>
-        <inertia ixx="1e-6" ixy="0" ixz="0" iyy="1e-6" iyz="0" izz="1e-6" />
+        <inertia ixx="1e-6" ixy="0" ixz="0" iyy="1e-6" iyz="0" izz="1e-6"/>
       </inertial>
     </link>

File: car_description/urdf/lidar.xacro (robot description, xacro)
@@ -4,5 +4,5 @@
   <xacro:macro name="lidar" params="name parent *origin">
     <joint name="${name}_joint" type="fixed">
-      <xacro:insert_block name="origin" />
+      <xacro:insert_block name="origin"/>
       <parent link="${parent}"/>
       <child link="${name}"/>
@@ -10,7 +10,7 @@
     <link name="${name}">
       <inertial>
-        <mass value="1e-5" />
+        <mass value="1e-5"/>
         <origin xyz="0 0 0" rpy="0 0 0"/>
-        <inertia ixx="1e-6" ixy="0" ixz="0" iyy="1e-6" iyz="0" izz="1e-6" />
+        <inertia ixx="1e-6" ixy="0" ixz="0" iyy="1e-6" iyz="0" izz="1e-6"/>
       </inertial>
     </link>

File: car_description/urdf/mondeo_dca/mondeo_dca.xacro (robot description, xacro)
@@ -1,8 +1,8 @@
 <?xml version="1.0"?>
-<robot name="mkz" xmlns:xacro="http://www.ros.org/wiki/xacro" >
+<robot name="mkz" xmlns:xacro="http://www.ros.org/wiki/xacro">
   <!-- Necessary includes -->
-  <xacro:include filename="$(find car_description)/urdf/mondeo_dca/mondeo_dca_params.xacro" />
-  <xacro:include filename="$(find car_description)/urdf/mondeo_dca/mondeo_dca_structure.xacro" />
+  <xacro:include filename="$(find car_description)/urdf/mondeo_dca/mondeo_dca_params.xacro"/>
+  <xacro:include filename="$(find car_description)/urdf/mondeo_dca/mondeo_dca_structure.xacro"/>
   <!-- Bolt-on sensors go here -->
-  <xacro:include filename="$(find car_description)/urdf/mondeo_dca/mondeo_dca_sensors.xacro" />
+  <xacro:include filename="$(find car_description)/urdf/mondeo_dca/mondeo_dca_sensors.xacro"/>
 </robot>

File: car_description/urdf/mondeo_dca/mondeo_dca_params.xacro (robot description, xacro)
@@ -2,50 +2,65 @@
 <robot xmlns:xacro="http://www.ros.org/wiki/xacro">
   <!-- CAR DIMENSIONS -->
-  <xacro:property name="car_length" value="4.8" />
-  <xacro:property name="car_width" value="1.75" />
-  <xacro:property name="car_height" value="1.5" />
-  <xacro:property name="car_offx" value="0.08" />
-  <xacro:property name="car_offy" value="0.0" />
-  <xacro:property name="car_offz" value="${0.04 + car_height/2}" />
-  <xacro:property name="centre_grav_z" value="0.0" /> <!-- Relative to base_link -->
-  <xacro:property name="vehicle_bonnet_x" value="${2.85 - base_link_x}" /> <!-- Relative to base_link -->
-  <xacro:property name="vehicle_bonnet_z" value="${0.69 - base_link_z}" /> <!-- Relative to base_link -->
-  <xacro:property name="front_axle_x" value="1.425" />
-  <xacro:property name="wheel_front_y" value="0.79121" /> <!-- The distance of front wheel joints from axle center -->
-  <xacro:property name="wheel_rear_y" value="0.7874" /> <!-- The distance of rear wheel joints from axle center -->
-  <xacro:property name="base_link_x" value="1.425" />
-  <xacro:property name="base_link_z" value="0.33" /> <!-- Above ground footprint -->
-  <xacro:property name="rear_axle_x" value="${-base_link_x}" /> <!-- Relative to base_link -->
-  <xacro:property name="rear_axle_z" value="0.0" /> <!-- Relative to base_link -->
-  <xacro:property name="roof_datum_x" value="1.88985" />
-  <xacro:property name="roof_datum_z" value="1.23242" />
-  <xacro:property name="front_bumper_x" value="0.915" /> <!-- Relative to vehicle_bonnet -->
-  <xacro:property name="front_bumper_z" value="${0.23 - (vehicle_bonnet_z + base_link_z)}" />
+  <xacro:property name="car_length" value="4.8"/>
+  <xacro:property name="car_width" value="1.75"/>
+  <xacro:property name="car_height" value="1.5"/>
+  <xacro:property name="car_offx" value="0.08"/>
+  <xacro:property name="car_offy" value="0.0"/>
+  <xacro:property name="car_offz" value="${0.04 + car_height/2}"/>
+  <xacro:property name="centre_grav_z" value="0.0"/>
+  <!-- Relative to base_link -->
+  <xacro:property name="vehicle_bonnet_x" value="${2.85 - base_link_x}"/>
+  <!-- Relative to base_link -->
+  <xacro:property name="vehicle_bonnet_z" value="${0.69 - base_link_z}"/>
+  <!-- Relative to base_link -->
+  <xacro:property name="front_axle_x" value="1.425"/>
+  <xacro:property name="wheel_front_y" value="0.79121"/>
+  <!-- The distance of front wheel joints from axle center -->
+  <xacro:property name="wheel_rear_y" value="0.7874"/>
+  <!-- The distance of rear wheel joints from axle center -->
+  <xacro:property name="base_link_x" value="1.425"/>
+  <xacro:property name="base_link_z" value="0.33"/>
+  <!-- Above ground footprint -->
+  <xacro:property name="rear_axle_x" value="${-base_link_x}"/>
+  <!-- Relative to base_link -->
+  <xacro:property name="rear_axle_z" value="0.0"/>
+  <!-- Relative to base_link -->
+  <xacro:property name="roof_datum_x" value="1.88985"/>
+  <xacro:property name="roof_datum_z" value="1.23242"/>
+  <xacro:property name="front_bumper_x" value="0.915"/>
+  <!-- Relative to vehicle_bonnet -->
+  <xacro:property name="front_bumper_z" value="${0.23 - (vehicle_bonnet_z + base_link_z)}"/>
   <!-- FOOTPRINT (Delimited by chassis extremes) -->
-  <xacro:property name="footprint_front_x" value="3.805" /> <!-- Relative to rear_axle -->
-  <xacro:property name="footprint_rear_x" value="-1.1" /> <!-- Relative to rear_axle -->
-  <xacro:property name="footprint_y" value="${2.14 / 2.0}" /> <!-- Symmetric about the centreline -->
+  <xacro:property name="footprint_front_x" value="3.805"/>
+  <!-- Relative to rear_axle -->
+  <xacro:property name="footprint_rear_x" value="-1.1"/>
+  <!-- Relative to rear_axle -->
+  <xacro:property name="footprint_y" value="${2.14 / 2.0}"/>
+  <!-- Symmetric about the centreline -->
   <!-- PHYSICAL PROPERTIES -->
-  <xacro:property name="wheel_side" value="0.785" />
-  <xacro:property name="wheel_width" value="0.2" />
-  <xacro:property name="wheel_radius" value="${0.66/2}" />
-  <xacro:property name="chassis_weight" value="1500" />
-  <xacro:property name="wheel_weight" value="10" />
+  <xacro:property name="wheel_side" value="0.785"/>
+  <xacro:property name="wheel_width" value="0.2"/>
+  <xacro:property name="wheel_radius" value="${0.66/2}"/>
+  <xacro:property name="chassis_weight" value="1500"/>
+  <xacro:property name="wheel_weight" value="10"/>
   <!-- SENSOR OFFSETS -->
-  <xacro:property name="oxts_x" value="${-0.59 - roof_datum_x}" /> <!-- Relative to roof_datum -->
-  <xacro:property name="oxts_y" value="-0.07" /> <!-- Relative to roof_datum -->
-  <xacro:property name="oxts_z" value="${0.9 - roof_datum_z - base_link_z}" /> <!-- Relative to roof_datum -->
+  <xacro:property name="oxts_x" value="${-0.59 - roof_datum_x}"/>
+  <!-- Relative to roof_datum -->
+  <xacro:property name="oxts_y" value="-0.07"/>
+  <!-- Relative to roof_datum -->
+  <xacro:property name="oxts_z" value="${0.9 - roof_datum_z - base_link_z}"/>
+  <!-- Relative to roof_datum -->
   <!-- The GPS antenna has been measured relative to the rear axle. The numerical values below gives these
        measurements. However, offsets are applied to make these values relative to the roof_datum -->
-  <xacro:property name="gps_antenna_base_left_x" value="${0.27 - roof_datum_x}" />
-  <xacro:property name="gps_antenna_base_left_y" value="0.5475" />
-  <xacro:property name="gps_antenna_base_left_z" value="${1.02 - roof_datum_z}" />
+  <xacro:property name="gps_antenna_base_left_x" value="${0.27 - roof_datum_x}"/>
+  <xacro:property name="gps_antenna_base_left_y" value="0.5475"/>
+  <xacro:property name="gps_antenna_base_left_z" value="${1.02 - roof_datum_z}"/>
   <!-- NOMENCLATURE -->
-  <xacro:property name="vehicle_bonnet" value="vehicle_bonnet" />
-  <xacro:property name="roof_datum" value="vehicle_roof_datum" />
-  <xacro:property name="footprint" value="footprint" />
-  <xacro:property name="lidar_top" value="lidar_top_mount" />
-  <xacro:property name="cham_left" value="camera_internal_left" />
-  <xacro:property name="cham_right" value="camera_internal_right" />
-  <xacro:property name="front_bumper" value="front_bumper" />
+  <xacro:property name="vehicle_bonnet" value="vehicle_bonnet"/>
+  <xacro:property name="roof_datum" value="vehicle_roof_datum"/>
+  <xacro:property name="footprint" value="footprint"/>
+  <xacro:property name="lidar_top" value="lidar_top_mount"/>
+  <xacro:property name="cham_left" value="camera_internal_left"/>
+  <xacro:property name="cham_right" value="camera_internal_right"/>
+  <xacro:property name="front_bumper" value="front_bumper"/>
 </robot>

File: car_description/urdf/mondeo_dca/mondeo_dca_sensors.xacro (robot description, xacro)
@@ -1,114 +1,114 @@
 <?xml version="1.0"?>
 <robot xmlns:xacro="http://www.ros.org/wiki/xacro">
-  <xacro:include filename="$(find car_description)/urdf/cameras.xacro" />
-  <xacro:include filename="$(find car_description)/urdf/lidar.xacro" />
-  <xacro:include filename="$(find car_description)/urdf/radar.xacro" />
-  <xacro:include filename="$(find car_description)/urdf/imu.xacro" />
-  <xacro:include filename="$(find car_description)/urdf/gps.xacro" />
-  <xacro:include filename="$(find car_description)/urdf/oxts.xacro" />
+  <xacro:include filename="$(find car_description)/urdf/cameras.xacro"/>
+  <xacro:include filename="$(find car_description)/urdf/lidar.xacro"/>
+  <xacro:include filename="$(find car_description)/urdf/radar.xacro"/>
+  <xacro:include filename="$(find car_description)/urdf/imu.xacro"/>
+  <xacro:include filename="$(find car_description)/urdf/gps.xacro"/>
+  <xacro:include filename="$(find car_description)/urdf/oxts.xacro"/>
   <!-- DCA ROOFBOX CAMERA MOUNTS -->
   <xacro:camera_mount name="camera_fsp_l_mount" parent="${roof_datum}">
-    <origin xyz="-0.11015 0.3 -0.06242" rpy="0 0.087266 0" />
+    <origin xyz="-0.11015 0.3 -0.06242" rpy="0 0.087266 0"/>
   </xacro:camera_mount>
   <xacro:camera_mount name="camera_fsp_r_mount" parent="${roof_datum}">
-    <origin xyz="-0.11015 -0.3 -0.06242" rpy="0 0.087266 0" />
+    <origin xyz="-0.11015 -0.3 -0.06242" rpy="0 0.087266 0"/>
   </xacro:camera_mount>
   <xacro:camera_mount name="camera_rsspf_l_mount" parent="${roof_datum}">
-    <origin xyz="-0.69015 -0.45 -0.00242" rpy="0 0.087266 -1.151917" />
+    <origin xyz="-0.69015 -0.45 -0.00242" rpy="0 0.087266 -1.151917"/>
   </xacro:camera_mount>
   <xacro:camera_mount name="camera_rsspf_r_mount" parent="${roof_datum}">
-    <origin xyz="-0.781503 -0.490673 -0.00242" rpy="0 0.087266 -1.151917" />
+    <origin xyz="-0.781503 -0.490673 -0.00242" rpy="0 0.087266 -1.151917"/>
   </xacro:camera_mount>
   <xacro:camera_mount name="camera_rsspr_l_mount" parent="${roof_datum}">
-    <origin xyz="-0.97015 -0.490673 -0.00242" rpy="0 0.087266 -1.989675" />
+    <origin xyz="-0.97015 -0.490673 -0.00242" rpy="0 0.087266 -1.989675"/>
   </xacro:camera_mount>
   <xacro:camera_mount name="camera_rsspr_r_mount" parent="${roof_datum}">
-    <origin xyz="-1.061503 -0.450 0.00242" rpy="0 0.087266 -1.989675" />
+    <origin xyz="-1.061503 -0.450 0.00242" rpy="0 0.087266 -1.989675"/>
   </xacro:camera_mount>
   <xacro:camera_mount name="camera_rsp_l_mount" parent="${roof_datum}">
-    <origin xyz="-1.11015 -0.3 0.00242" rpy="0 0.087266 3.141592654" />
+    <origin xyz="-1.11015 -0.3 0.00242" rpy="0 0.087266 3.141592654"/>
   </xacro:camera_mount>
   <xacro:camera_mount name="camera_rsp_r_mount" parent="${roof_datum}">
-    <origin xyz="-1.11015 0.3 0.00242" rpy="0 0.087266 3.141592654" />
+    <origin xyz="-1.11015 0.3 0.00242" rpy="0 0.087266 3.141592654"/>
   </xacro:camera_mount>
   <xacro:camera_mount name="camera_lsspr_l_mount" parent="${roof_datum}">
-    <origin xyz="-1.061503 0.450 0.00242" rpy="0 0.087266 1.989675" />
+    <origin xyz="-1.061503 0.450 0.00242" rpy="0 0.087266 1.989675"/>
   </xacro:camera_mount>
   <xacro:camera_mount name="camera_lsspr_r_mount" parent="${roof_datum}">
-    <origin xyz="-0.97015 0.490673 -0.00242" rpy="0 0.087266 1.989675" />
+    <origin xyz="-0.97015 0.490673 -0.00242" rpy="0 0.087266 1.989675"/>
   </xacro:camera_mount>
   <xacro:camera_mount name="camera_lsspf_l_mount" parent="${roof_datum}">
-    <origin xyz="-0.781503 0.490673 -0.00242" rpy="0 0.087266 1.151917" />
+    <origin xyz="-0.781503 0.490673 -0.00242" rpy="0 0.087266 1.151917"/>
   </xacro:camera_mount>
   <xacro:camera_mount name="camera_lsspf_r_mount" parent="${roof_datum}">
-    <origin xyz="-0.69015 0.45 -0.00242" rpy="0 0.087266 1.151917" />
+    <origin xyz="-0.69015 0.45 -0.00242" rpy="0 0.087266 1.151917"/>
   </xacro:camera_mount>
   <xacro:camera_mount name="camera_tele1_mount" parent="${roof_datum}">
-    <origin xyz="-0.11015 -0.120 -0.06242" rpy="0 0 0" />
+    <origin xyz="-0.11015 -0.120 -0.06242" rpy="0 0 0"/>
   </xacro:camera_mount>
   <xacro:camera_mount name="camera_tele2_mount" parent="${roof_datum}">
-    <origin xyz="-0.11015 -0.205 -0.06242" rpy="0 0 0" />
+    <origin xyz="-0.11015 -0.205 -0.06242" rpy="0 0 0"/>
   </xacro:camera_mount>
   <xacro:camera_mount name="camera_ir1_mount" parent="${roof_datum}">
-    <origin xyz="-0.11015 0.120 -0.06242" rpy="0 0 0" />
+    <origin xyz="-0.11015 0.120 -0.06242" rpy="0 0 0"/>
   </xacro:camera_mount>
   <xacro:camera_mount name="camera_ir2_mount" parent="${roof_datum}">
-    <origin xyz="-0.11015 0.205 -0.06242" rpy="0 0 0" />
+    <origin xyz="-0.11015 0.205 -0.06242" rpy="0 0 0"/>
   </xacro:camera_mount>
   <!-- IMU -->
   <xacro:imu imu="imu_rear_mount">
-    <origin xyz="${oxts_x-0.19} ${oxts_y+0.23} ${oxts_z-0.44}" rpy="0 0 0" />
+    <origin xyz="${oxts_x-0.19} ${oxts_y+0.23} ${oxts_z-0.44}" rpy="0 0 0"/>
   </xacro:imu>
   <xacro:imu imu="imu_fsp_r_mount">
-    <origin xyz="-0.23515 -0.355 -0.05442" rpy="0 0 0" />
+    <origin xyz="-0.23515 -0.355 -0.05442" rpy="0 0 0"/>
   </xacro:imu>
   <!-- OXTS -->
   <xacro:oxts name="oxts">
-    <origin xyz="${oxts_x} ${oxts_y} ${oxts_z}" rpy="0.0 0.0 0.0" />
+    <origin xyz="${oxts_x} ${oxts_y} ${oxts_z}" rpy="0.0 0.0 0.0"/>
   </xacro:oxts>
   <!-- GPS -->
   <xacro:gps name="gps_antenna_right_mount">
-    <origin xyz="${gps_antenna_base_left_x} ${-gps_antenna_base_left_y} ${gps_antenna_base_left_z}" rpy="0 0 0" />
+    <origin xyz="${gps_antenna_base_left_x} ${-gps_antenna_base_left_y} ${gps_antenna_base_left_z}" rpy="0 0 0"/>
   </xacro:gps>
   <xacro:gps name="gps_antenna_left_mount">
-    <origin xyz="${gps_antenna_base_left_x} ${gps_antenna_base_left_y} ${gps_antenna_base_left_z}" rpy="0 0 0" />
+    <origin xyz="${gps_antenna_base_left_x} ${gps_antenna_base_left_y} ${gps_antenna_base_left_z}" rpy="0 0 0"/>
   </xacro:gps>
   <!-- LIDAR -->
   <xacro:lidar name="lidar_top" parent="${roof_datum}">
-    <origin xyz="-0.66015 0 0.19758" rpy="0 0 0" />
+    <origin xyz="-0.66015 0 0.19758" rpy="0 0 0"/>
   </xacro:lidar>
   <xacro:lidar name="lidar_left" parent="${roof_datum}">
-    <origin xyz="-0.03015 0.720 -0.22242" rpy="-0.087266 0.087266 0.6562438" />
+    <origin xyz="-0.03015 0.720 -0.22242" rpy="-0.087266 0.087266 0.6562438"/>
   </xacro:lidar>
   <xacro:lidar name="lidar_right" parent="${roof_datum}">
-    <origin xyz="-0.03015 -0.720 -0.22242" rpy="0.087266 0.087266 -0.6562438" />
+    <origin xyz="-0.03015 -0.720 -0.22242" rpy="0.087266 0.087266 -0.6562438"/>
   </xacro:lidar>
   <xacro:lidar name="lidar_ouster_top" parent="${roof_datum}">
-    <origin xyz="-0.65855 0 0.21849" rpy="0 -0.017453 0" />
+    <origin xyz="-0.65855 0 0.21849" rpy="0 -0.017453 0"/>
   </xacro:lidar>
   <!-- RADAR -->
   <xacro:radar name="radar_roof_left_front_mount" parent="${roof_datum}">
-    <origin xyz="-0.30185 0.48847 -0.02042" rpy="3.141592654 0 1.33657" />
+    <origin xyz="-0.30185 0.48847 -0.02042" rpy="3.141592654 0 1.33657"/>
   </xacro:radar>
   <xacro:radar name="radar_roof_right_front_mount" parent="${roof_datum}">
-    <origin xyz="-0.30185 -0.48847 -0.02042" rpy="0 0 -1.31605" />
+    <origin xyz="-0.30185 -0.48847 -0.02042" rpy="0 0 -1.31605"/>
   </xacro:radar>
   <xacro:radar name="radar_roof_left_rear_mount" parent="${roof_datum}">
-    <origin xyz="-1.12515 0.410 0.00258" rpy="0 0 2.3658" />
+    <origin xyz="-1.12515 0.410 0.00258" rpy="0 0 2.3658"/>
   </xacro:radar>
   <xacro:radar name="radar_roof_right_rear_mount" parent="${roof_datum}">
-    <origin xyz="-1.12515 -0.410 0.00258" rpy="3.141592654 0 -2.3606" />
+    <origin xyz="-1.12515 -0.410 0.00258" rpy="3.141592654 0 -2.3606"/>
   </xacro:radar>
   <xacro:radar name="radar_bumper_front_left_mount" parent="${front_bumper}">
-    <origin xyz="-0.16666 0.58893 0.24618" rpy="0 0 0.645772" />
+    <origin xyz="-0.16666 0.58893 0.24618" rpy="0 0 0.645772"/>
   </xacro:radar>
   <xacro:radar name="radar_bumper_front_centre_mount" parent="${front_bumper}">
-    <origin xyz="-0.07709 0 0.34618" rpy="0 0 0" />
+    <origin xyz="-0.07709 0 0.34618" rpy="0 0 0"/>
   </xacro:radar>
   <xacro:radar name="radar_bumper_front_right_mount" parent="${front_bumper}">
-    <origin xyz="-0.16666 -0.58893 0.24618" rpy="3.141592654 0 -0.645772" />
+    <origin xyz="-0.16666 -0.58893 0.24618" rpy="3.141592654 0 -0.645772"/>
   </xacro:radar>
   <xacro:radar name="radar_bumper_rear_centre_mount" parent="rear_axle">
-    <origin xyz="-1.04 0 0.16" rpy="0 0 3.141592654" />
+    <origin xyz="-1.04 0 0.16" rpy="0 0 3.141592654"/>
   </xacro:radar>
 </robot>
