Commit message: Fix pre-commit linting, advice and suggestions

File: car_description/urdf/mondeo_dca/mondeo_dca_structure.xacro (robot description, xacro)
@@ -1,14 +1,17 @@
 <?xml version="1.0"?>
-<robot xmlns:xacro="http://www.ros.org/wiki/xacro" name="dbw_mkz" >
-  <link name="base_footprint">
-  </link>
+<robot xmlns:xacro="http://www.ros.org/wiki/xacro" name="dbw_mkz">
+  <link name="base_footprint"/>
   <link name="base_link">
     <inertial>
       <origin xyz="0 0 ${centre_grav_z}" rpy="0 0 0"/>
       <mass value="${chassis_weight}"/>
-        <inertia
-        ixx="${(chassis_weight/12)*((car_width**2)+(car_height**2))}" ixy="0.0" ixz="0.0"
-        iyy="${(chassis_weight/12)*((car_width**2)+(car_length**2))}" iyz="0.0"
-        izz="${(chassis_weight/12)*((car_height**2)+(car_length**2))}"/>
+      <inertia
+        ixx="${(chassis_weight/12)*((car_width**2)+(car_height**2))}"
+        ixy="0.0"
+        ixz="0.0"
+        iyy="${(chassis_weight/12)*((car_width**2)+(car_length**2))}"
+        iyz="0.0"
+        izz="${(chassis_weight/12)*((car_height**2)+(car_length**2))}"
+      />
     </inertial>
     <visual name="chassis">
@@ -35,8 +38,5 @@
       <origin xyz="0 0 0" rpy="0 0 0"/>
       <mass value="0.01"/>
-      <inertia
-        ixx="0.1" ixy="0.0" ixz="0.0"
-        iyy="0.1" iyz="0.0"
-        izz="0.1"/>
+      <inertia ixx="0.1" ixy="0.0" ixz="0.0" iyy="0.1" iyz="0.0" izz="0.1"/>
     </inertial>
   </link>
@@ -50,8 +50,5 @@
       <origin xyz="0 0 0" rpy="0 0 0"/>
       <mass value="0.01"/>
-      <inertia
-        ixx="0.1" ixy="0.0" ixz="0.0"
-        iyy="0.1" iyz="0.0"
-        izz="0.1"/>
+      <inertia ixx="0.1" ixy="0.0" ixz="0.0" iyy="0.1" iyz="0.0" izz="0.1"/>
     </inertial>
   </link>
@@ -65,8 +62,5 @@
       <origin xyz="0 0 0" rpy="0 0 0"/>
       <mass value="0.01"/>
-      <inertia
-        ixx="0.1" ixy="0.0" ixz="0.0"
-        iyy="0.1" iyz="0.0"
-        izz="0.1"/>
+      <inertia ixx="0.1" ixy="0.0" ixz="0.0" iyy="0.1" iyz="0.0" izz="0.1"/>
     </inertial>
   </link>
@@ -90,7 +84,11 @@
       <mass value="${wheel_weight}"/>
       <inertia
-        ixx="${(wheel_weight/12)*(3*(wheel_radius**2)+(wheel_width**2))}" ixy="0.0" ixz="0.0"
-        iyy="${(wheel_weight/12)*(3*(wheel_radius**2)+(wheel_width**2))}" iyz="0.0"
-        izz="${(wheel_weight*(wheel_radius**2))/2}" />
+        ixx="${(wheel_weight/12)*(3*(wheel_radius**2)+(wheel_width**2))}"
+        ixy="0.0"
+        ixz="0.0"
+        iyy="${(wheel_weight/12)*(3*(wheel_radius**2)+(wheel_width**2))}"
+        iyz="0.0"
+        izz="${(wheel_weight*(wheel_radius**2))/2}"
+      />
     </inertial>
     <visual name="wheel_fl_visual">
@@ -103,15 +101,15 @@
     <collision name="wheel_fl_collision">
       <origin xyz="0 0 0" rpy="0 0 0"/>
-        <geometry>
-          <sphere radius="${wheel_radius}"/>
-        </geometry>
-        <surface>
-          <friction>
-            <ode>
-              <mu>1.2</mu>
-              <mu2>1.2</mu2>
-            </ode>
-          </friction>
-        </surface>
+      <geometry>
+        <sphere radius="${wheel_radius}"/>
+      </geometry>
+      <surface>
+        <friction>
+          <ode>
+            <mu>1.2</mu>
+            <mu2>1.2</mu2>
+          </ode>
+        </friction>
+      </surface>
     </collision>
   </link>
@@ -121,7 +119,11 @@
       <mass value="${wheel_weight}"/>
       <inertia
-        ixx="${(wheel_weight/12)*(3*(wheel_radius**2)+(wheel_width**2))}" ixy="0.0" ixz="0.0"
-        iyy="${(wheel_weight/12)*(3*(wheel_radius**2)+(wheel_width**2))}" iyz="0.0"
-        izz="${(wheel_weight*(wheel_radius**2))/2}" />
+        ixx="${(wheel_weight/12)*(3*(wheel_radius**2)+(wheel_width**2))}"
+        ixy="0.0"
+        ixz="0.0"
+        iyy="${(wheel_weight/12)*(3*(wheel_radius**2)+(wheel_width**2))}"
+        iyz="0.0"
+        izz="${(wheel_weight*(wheel_radius**2))/2}"
+      />
     </inertial>
     <visual name="wheel_fr_visual">
@@ -134,15 +136,15 @@
     <collision name="wheel_fr_collision">
       <origin xyz="0 0 0" rpy="0 0 0"/>
-        <geometry>
-          <sphere radius="${wheel_radius}"/>
-        </geometry>
-        <surface>
-          <friction>
-            <ode>
-              <mu>1.2</mu>
-              <mu2>1.2</mu2>
-            </ode>
-          </friction>
-        </surface>
+      <geometry>
+        <sphere radius="${wheel_radius}"/>
+      </geometry>
+      <surface>
+        <friction>
+          <ode>
+            <mu>1.2</mu>
+            <mu2>1.2</mu2>
+          </ode>
+        </friction>
+      </surface>
     </collision>
   </link>
@@ -152,7 +154,11 @@
       <mass value="${wheel_weight}"/>
       <inertia
-        ixx="${(wheel_weight/12)*(3*(wheel_radius**2)+(wheel_width**2))}" ixy="0.0" ixz="0.0"
-        iyy="${(wheel_weight/12)*(3*(wheel_radius**2)+(wheel_width**2))}" iyz="0.0"
-        izz="${(wheel_weight*(wheel_radius**2))/2}" />
+        ixx="${(wheel_weight/12)*(3*(wheel_radius**2)+(wheel_width**2))}"
+        ixy="0.0"
+        ixz="0.0"
+        iyy="${(wheel_weight/12)*(3*(wheel_radius**2)+(wheel_width**2))}"
+        iyz="0.0"
+        izz="${(wheel_weight*(wheel_radius**2))/2}"
+      />
     </inertial>
     <visual name="wheel_rl_visual">
@@ -165,15 +171,15 @@
     <collision name="wheel_rl_collision">
       <origin xyz="0 0 0" rpy="0 0 0"/>
-        <geometry>
-          <sphere radius="${wheel_radius}"/>
-        </geometry>
-        <surface>
-          <friction>
-            <ode>
-              <mu>1.2</mu>
-              <mu2>1.2</mu2>
-            </ode>
-          </friction>
-        </surface>
+      <geometry>
+        <sphere radius="${wheel_radius}"/>
+      </geometry>
+      <surface>
+        <friction>
+          <ode>
+            <mu>1.2</mu>
+            <mu2>1.2</mu2>
+          </ode>
+        </friction>
+      </surface>
     </collision>
   </link>
@@ -183,7 +189,11 @@
       <mass value="${wheel_weight}"/>
       <inertia
-        ixx="${(wheel_weight/12)*(3*(wheel_radius**2)+(wheel_width**2))}" ixy="0.0" ixz="0.0"
-        iyy="${(wheel_weight/12)*(3*(wheel_radius**2)+(wheel_width**2))}" iyz="0.0"
-        izz="${(wheel_weight*(wheel_radius**2))/2}" />
+        ixx="${(wheel_weight/12)*(3*(wheel_radius**2)+(wheel_width**2))}"
+        ixy="0.0"
+        ixz="0.0"
+        iyy="${(wheel_weight/12)*(3*(wheel_radius**2)+(wheel_width**2))}"
+        iyz="0.0"
+        izz="${(wheel_weight*(wheel_radius**2))/2}"
+      />
     </inertial>
     <visual name="wheel_rr_visual">
@@ -196,15 +206,15 @@
     <collision name="wheel_rr_collision">
       <origin xyz="0 0 0" rpy="0 0 0"/>
-        <geometry>
-          <sphere radius="${wheel_radius}"/>
-        </geometry>
-        <surface>
-          <friction>
-            <ode>
-              <mu>1.2</mu>
-              <mu2>1.2</mu2>
-            </ode>
-          </friction>
-        </surface>
+      <geometry>
+        <sphere radius="${wheel_radius}"/>
+      </geometry>
+      <surface>
+        <friction>
+          <ode>
+            <mu>1.2</mu>
+            <mu2>1.2</mu2>
+          </ode>
+        </friction>
+      </surface>
     </collision>
   </link>
@@ -218,8 +228,5 @@
       <origin xyz="0 0 0" rpy="0 0 0"/>
       <mass value="0.01"/>
-      <inertia
-        ixx="0.1" ixy="0.0" ixz="0.0"
-        iyy="0.1" iyz="0.0"
-        izz="0.1"/>
+      <inertia ixx="0.1" ixy="0.0" ixz="0.0" iyy="0.1" iyz="0.0" izz="0.1"/>
     </inertial>
   </link>
@@ -233,8 +240,5 @@
       <origin xyz="0 0 0" rpy="0 0 0"/>
       <mass value="0.01"/>
-      <inertia
-        ixx="0.1" ixy="0.0" ixz="0.0"
-        iyy="0.1" iyz="0.0"
-        izz="0.1"/>
+      <inertia ixx="0.1" ixy="0.0" ixz="0.0" iyy="0.1" iyz="0.0" izz="0.1"/>
     </inertial>
   </link>
@@ -263,5 +267,6 @@
     <child link="wheel_fl"/>
     <axis xyz="0 0 1.0"/>
-    <limit dissipation="1" effort="1000.0" velocity="${48*pi}"/> <!-- ~40mph -->
+    <limit dissipation="1" effort="1000.0" velocity="${48*pi}"/>
+    <!-- ~40mph -->
   </joint>
   <joint name="wheel_fr" type="continuous">
@@ -270,5 +275,6 @@
     <child link="wheel_fr"/>
     <axis xyz="0 0 1.0"/>
-    <limit dissipation="1" effort="1000.0" velocity="${48*pi}"/> <!-- ~40mph -->
+    <limit dissipation="1" effort="1000.0" velocity="${48*pi}"/>
+    <!-- ~40mph -->
   </joint>
   <joint name="wheel_rl" type="continuous">
@@ -277,5 +283,6 @@
     <child link="wheel_rl"/>
     <axis xyz="0 0 1.0"/>
-    <limit dissipation="1" effort="1000.0" velocity="${48*pi}"/> <!-- ~40mph -->
+    <limit dissipation="1" effort="1000.0" velocity="${48*pi}"/>
+    <!-- ~40mph -->
   </joint>
   <joint name="wheel_rr" type="continuous">
@@ -284,5 +291,6 @@
     <child link="wheel_rr"/>
     <axis xyz="0 0 1.0"/>
-    <limit dissipation="1" effort="1000.0" velocity="${48*pi}"/> <!-- ~40mph -->
+    <limit dissipation="1" effort="1000.0" velocity="${48*pi}"/>
+    <!-- ~40mph -->
   </joint>
   <!-- Footprint Frames -->

File: car_description/urdf/oxts.xacro (robot description, xacro)
@@ -3,5 +3,5 @@
   <xacro:macro name="oxts" params="name *origin">
     <joint name="${name}_joint" type="fixed">
-      <xacro:insert_block name="origin" />
+      <xacro:insert_block name="origin"/>
       <parent link="${roof_datum}"/>
       <child link="${name}"/>
@@ -9,7 +9,7 @@
     <link name="${name}">
       <inertial>
-        <mass value="1e-5" />
+        <mass value="1e-5"/>
         <origin xyz="0 0 0" rpy="0 0 0"/>
-        <inertia ixx="1e-6" ixy="0" ixz="0" iyy="1e-6" iyz="0" izz="1e-6" />
+        <inertia ixx="1e-6" ixy="0" ixz="0" iyy="1e-6" iyz="0" izz="1e-6"/>
       </inertial>
     </link>

File: car_description/urdf/radar.xacro (robot description, xacro)
@@ -3,5 +3,5 @@
   <xacro:macro name="radar" params="name parent *origin">
     <joint name="${name}_joint" type="fixed">
-      <xacro:insert_block name="origin" />
+      <xacro:insert_block name="origin"/>
       <parent link="${parent}"/>
       <child link="${name}"/>
@@ -9,7 +9,7 @@
     <link name="${name}">
       <inertial>
-        <mass value="1e-5" />
+        <mass value="1e-5"/>
         <origin xyz="0 0 0" rpy="0 0 0"/>
-        <inertia ixx="1e-6" ixy="0" ixz="0" iyy="1e-6" iyz="0" izz="1e-6" />
+        <inertia ixx="1e-6" ixy="0" ixz="0" iyy="1e-6" iyz="0" izz="1e-6"/>
       </inertial>
     </link>

File: car_description/urdf/velodyne/HDL-32E.urdf.xacro (robot description, xacro)
@@ -4,8 +4,11 @@
   to avoid having to install the Velodyne meshes -->
 <robot xmlns:xacro="http://www.ros.org/wiki/xacro" name="HDL-32E">
-  <xacro:property name="M_PI" value="3.1415926535897931" />
-  <xacro:macro name="HDL-32E" params="*origin parent:=base_link name:=velodyne topic:=/velodyne_points hz:=10 lasers:=32 samples:=2187 collision_range:=0.3 min_range:=0.9 max_range:=130.0 noise:=0.008 min_angle:=-${M_PI} max_angle:=${M_PI} gpu:=false">
+  <xacro:property name="M_PI" value="3.1415926535897931"/>
+  <xacro:macro
+    name="HDL-32E"
+    params="*origin parent:=base_link name:=velodyne topic:=/velodyne_points hz:=10 lasers:=32 samples:=2187 collision_range:=0.3 min_range:=0.9 max_range:=130.0 noise:=0.008 min_angle:=-${M_PI} max_angle:=${M_PI} gpu:=false"
+  >
     <joint name="${name}_base_mount_joint" type="fixed">
-      <xacro:insert_block name="origin" />
+      <xacro:insert_block name="origin"/>
       <parent link="${parent}"/>
       <child link="${name}_base_link"/>
@@ -15,11 +18,16 @@
         <mass value="1.0"/>
         <origin xyz="0 0 0.07212"/>
-        <inertia ixx="${(1.0 * (3.0*0.04267*0.04267 + 0.14424*0.14424)) / 12.0}" ixy="0" ixz="0"
-          iyy="${(1.0 * (3.0*0.04267*0.04267 + 0.14424*0.14424)) / 12.0}" iyz="0"
-          izz="${0.5 * 1.0 * (0.04267*0.04267)}"/>
+        <inertia
+          ixx="${(1.0 * (3.0*0.04267*0.04267 + 0.14424*0.14424)) / 12.0}"
+          ixy="0"
+          ixz="0"
+          iyy="${(1.0 * (3.0*0.04267*0.04267 + 0.14424*0.14424)) / 12.0}"
+          iyz="0"
+          izz="${0.5 * 1.0 * (0.04267*0.04267)}"
+        />
       </inertial>
       <visual>
         <geometry>
-          <mesh filename="package://velodyne_description/meshes/HDL32E_base.dae" />
+          <mesh filename="package://velodyne_description/meshes/HDL32E_base.dae"/>
         </geometry>
       </visual>
@@ -31,7 +39,7 @@
       </collision>
     </link>
-    <joint name="${name}_base_scan_joint" type="fixed" >
-      <origin xyz="0 0 0.09081" rpy="0 0 0" />
-      <parent link="${name}_base_link" />
+    <joint name="${name}_base_scan_joint" type="fixed">
+      <origin xyz="0 0 0.09081" rpy="0 0 0"/>
+      <parent link="${name}_base_link"/>
       <child link="${name}"/>
     </joint>
@@ -43,7 +51,7 @@
       </inertial>
       <visual>
-        <origin xyz="0 0 -0.09081" rpy="0 0 0" />
+        <origin xyz="0 0 -0.09081" rpy="0 0 0"/>
         <geometry>
-          <mesh filename="package://velodyne_description/meshes/HDL32E_scan.dae" />
+          <mesh filename="package://velodyne_description/meshes/HDL32E_scan.dae"/>
         </geometry>
       </visual>
@@ -68,5 +76,5 @@
                 <resolution>1</resolution>
                 <min_angle>-${30.67*M_PI/180.0}</min_angle>
-                <max_angle> ${10.67*M_PI/180.0}</max_angle>
+                <max_angle>${10.67*M_PI/180.0}</max_angle>
               </vertical>
             </scan>
@@ -108,5 +116,5 @@
                 <resolution>1</resolution>
                 <min_angle>-${30.67*M_PI/180.0}</min_angle>
-                <max_angle> ${10.67*M_PI/180.0}</max_angle>
+                <max_angle>${10.67*M_PI/180.0}</max_angle>
               </vertical>
             </scan>
