Commit message: Fix IMUs and GPS antennas TFs
- Fix `imu_rear_mount` and `imu_fsp_r_mount` to align with
  imu driver measurements
- Add `gps_antenna_*_sensor` frame to align with current
  mounting.

File: av_car_description/urdf/gps.xacro (robot description, xacro)
@@ -1,8 +1,8 @@
 <?xml version="1.0"?>
 <robot xmlns:xacro="http://www.ros.org/wiki/xacro">
-  <xacro:macro name="gps" params="name *origin">
+  <xacro:macro name="gps" params="name parent *origin">
     <joint name="${name}_joint" type="fixed">
       <xacro:insert_block name="origin"/>
-      <parent link="${roof_datum}"/>
+      <parent link="${parent}"/>
       <child link="${name}"/>
     </joint>

File: av_car_description/urdf/mondeo_dca/mondeo_dca_sensors.xacro (robot description, xacro)
@@ -130,8 +130,8 @@
   <!-- IMU -->
   <xacro:imu imu="imu_rear_mount">
-    <origin xyz="${oxts_x-0.19} ${oxts_y+0.23} ${oxts_z-0.44}" rpy="0 0 0"/>
+    <origin xyz="${oxts_x-0.19} ${oxts_y+0.23} ${oxts_z-0.44}" rpy="0 0 1.5708"/>
   </xacro:imu>
   <xacro:imu imu="imu_fsp_r_mount">
-    <origin xyz="-0.23515 -0.355 -0.05442" rpy="0 0 0"/>
+    <origin xyz="-0.23515 -0.355 -0.05442" rpy="0 0 1.5708"/>
   </xacro:imu>
   <!-- OXTS -->
@@ -140,9 +140,15 @@
   </xacro:oxts>
   <!-- GPS -->
-  <xacro:gps name="gps_antenna_right_mount">
+  <xacro:gps name="gps_antenna_right_mount" parent="${roof_datum}">
     <origin xyz="${gps_antenna_base_left_x} ${-gps_antenna_base_left_y} ${gps_antenna_base_left_z}" rpy="0 0 0"/>
   </xacro:gps>
-  <xacro:gps name="gps_antenna_left_mount">
+  <xacro:gps name="gps_antenna_right_sensor" parent="gps_antenna_right_mount">
+    <origin xyz="-1.1 0.0 0.0" rpy="0 0 0"/>
+  </xacro:gps>
+  <xacro:gps name="gps_antenna_left_mount" parent="${roof_datum}">
     <origin xyz="${gps_antenna_base_left_x} ${gps_antenna_base_left_y} ${gps_antenna_base_left_z}" rpy="0 0 0"/>
+  </xacro:gps>
+  <xacro:gps name="gps_antenna_left_sensor" parent="gps_antenna_left_mount">
+    <origin xyz="-1.1 0.0 0.0" rpy="0 0 0"/>
   </xacro:gps>
   <!-- LIDAR -->
