Commit message: Rename pkgs name and references

File: av_lxo_description/urdf/lidar.xacro (robot description, xacro)
@@ -1,5 +1,5 @@
 <?xml version="1.0"?>
 <robot xmlns:xacro="http://www.ros.org/wiki/xacro">
-  <xacro:include filename="$(find av_car_description)/urdf/velodyne/HDL-32E.urdf.xacro"/>
+  <xacro:include filename="$(find av_lxo_description)/urdf/velodyne/HDL-32E.urdf.xacro"/>
   <xacro:macro name="lidar" params="name parent *origin">
     <joint name="${name}_joint" type="fixed">

File: av_lxo_description/urdf/mondeo_dca/mondeo_dca.xacro (robot description, xacro)
@@ -2,7 +2,7 @@
 <robot name="mkz" xmlns:xacro="http://www.ros.org/wiki/xacro">
   <!-- Necessary includes -->
-  <xacro:include filename="$(find av_car_description)/urdf/mondeo_dca/mondeo_dca_params.xacro"/>
-  <xacro:include filename="$(find av_car_description)/urdf/mondeo_dca/mondeo_dca_structure.xacro"/>
+  <xacro:include filename="$(find av_lxo_description)/urdf/mondeo_dca/mondeo_dca_params.xacro"/>
+  <xacro:include filename="$(find av_lxo_description)/urdf/mondeo_dca/mondeo_dca_structure.xacro"/>
   <!-- Bolt-on sensors go here -->
-  <xacro:include filename="$(find av_car_description)/urdf/mondeo_dca/mondeo_dca_sensors.xacro"/>
+  <xacro:include filename="$(find av_lxo_description)/urdf/mondeo_dca/mondeo_dca_sensors.xacro"/>
 </robot>

File: av_lxo_description/urdf/mondeo_dca/mondeo_dca_sensors.xacro (robot description, xacro)
@@ -1,10 +1,10 @@
 <?xml version="1.0"?>
 <robot xmlns:xacro="http://www.ros.org/wiki/xacro">
-  <xacro:include filename="$(find av_car_description)/urdf/cameras.xacro"/>
-  <xacro:include filename="$(find av_car_description)/urdf/lidar.xacro"/>
-  <xacro:include filename="$(find av_car_description)/urdf/radar.xacro"/>
-  <xacro:include filename="$(find av_car_description)/urdf/imu.xacro"/>
-  <xacro:include filename="$(find av_car_description)/urdf/gps.xacro"/>
-  <xacro:include filename="$(find av_car_description)/urdf/oxts.xacro"/>
+  <xacro:include filename="$(find av_lxo_description)/urdf/cameras.xacro"/>
+  <xacro:include filename="$(find av_lxo_description)/urdf/lidar.xacro"/>
+  <xacro:include filename="$(find av_lxo_description)/urdf/radar.xacro"/>
+  <xacro:include filename="$(find av_lxo_description)/urdf/imu.xacro"/>
+  <xacro:include filename="$(find av_lxo_description)/urdf/gps.xacro"/>
+  <xacro:include filename="$(find av_lxo_description)/urdf/oxts.xacro"/>
   <!-- DCA ROOFBOX CAMERA MOUNTS -->
   <xacro:camera_mount name="camera_fsp_l_mount" parent="${roof_datum}">

File: av_lxo_description/urdf/mondeo_dca/mondeo_dca_structure.xacro (robot description, xacro)
@@ -18,5 +18,5 @@
       <origin xyz="${1.361 - base_link_x} 0 -0.33647" rpy="0 0 ${pi/2}"/>
       <geometry>
-        <mesh filename="package://av_car_meshes/meshes/mondeo_grey.dae" scale="1 1 1"/>
+        <mesh filename="package://av_lxo_meshes/meshes/mondeo_grey.dae" scale="1 1 1"/>
       </geometry>
       <material name="black.001"/>
@@ -25,5 +25,5 @@
       <origin xyz="${1.4621 - base_link_x} -0.03046 0.350609" rpy="${pi/2} 0 -${pi}"/>
       <geometry>
-        <mesh filename="package://av_car_meshes/meshes/body_collision.stl" scale="0.001 0.001 0.001"/>
+        <mesh filename="package://av_lxo_meshes/meshes/body_collision.stl" scale="0.001 0.001 0.001"/>
       </geometry>
     </collision>
@@ -95,5 +95,5 @@
       <origin xyz="0 0 0" rpy="-${pi/2} ${pi/2} 0"/>
       <geometry>
-        <mesh filename="package://av_car_meshes/meshes/mondeo_wheel.dae"/>
+        <mesh filename="package://av_lxo_meshes/meshes/mondeo_wheel.dae"/>
       </geometry>
       <material name="carpaint_002"/>
@@ -130,5 +130,5 @@
       <origin xyz="0 0 0" rpy="-${pi/2} -${pi/2} 0"/>
       <geometry>
-        <mesh filename="package://av_car_meshes/meshes/mondeo_wheel.dae"/>
+        <mesh filename="package://av_lxo_meshes/meshes/mondeo_wheel.dae"/>
       </geometry>
       <material name="carpaint_002.001"/>
@@ -165,5 +165,5 @@
       <origin xyz="0 0 0" rpy="-${pi/2} ${pi/2} 0"/>
       <geometry>
-        <mesh filename="package://av_car_meshes/meshes/mondeo_wheel.dae"/>
+        <mesh filename="package://av_lxo_meshes/meshes/mondeo_wheel.dae"/>
       </geometry>
       <material name="carpaint_002.003"/>
@@ -200,5 +200,5 @@
       <origin xyz="0 0 0" rpy="-${pi/2} -${pi/2} 0"/>
       <geometry>
-        <mesh filename="package://av_car_meshes/meshes/mondeo_wheel.dae"/>
+        <mesh filename="package://av_lxo_meshes/meshes/mondeo_wheel.dae"/>
       </geometry>
       <material name="carpaint_002.002"/>
