Commit message: Set rear_axle as gloabl reference
- Rename base_link to center_axle
- Adjust parameters to keep consistency

File: av_lxo_description/urdf/mondeo_dca/mondeo_dca_params.xacro (robot description, xacro)
@@ -9,26 +9,25 @@
   <xacro:property name="car_offz" value="${0.04 + car_height/2}"/>
   <xacro:property name="centre_grav_z" value="0.0"/>
-  <!-- Relative to base_link -->
-  <xacro:property name="vehicle_bonnet_x" value="${2.85 - base_link_x}"/>
-  <!-- Relative to base_link -->
-  <xacro:property name="vehicle_bonnet_z" value="${0.69 - base_link_z}"/>
-  <!-- Relative to base_link -->
-  <xacro:property name="front_axle_x" value="1.425"/>
+  <xacro:property name="wheelbase" value="2.85"/>
+  <!-- Relative to rear_axle -->
+  <xacro:property name="vehicle_bonnet_x" value="${wheelbase}"/>
+  <!-- Relative to rear_axle -->
+  <xacro:property name="vehicle_bonnet_z" value="${0.69 - center_axle_z}"/>
+  <!-- Relative to rear_axle -->
+  <xacro:property name="front_axle_x" value="${wheelbase}"/>
   <xacro:property name="wheel_front_y" value="0.79121"/>
   <!-- The distance of front wheel joints from axle center -->
   <xacro:property name="wheel_rear_y" value="0.7874"/>
   <!-- The distance of rear wheel joints from axle center -->
-  <xacro:property name="base_link_x" value="1.425"/>
-  <xacro:property name="base_link_z" value="0.33"/>
+  <xacro:property name="center_axle_x" value="1.425"/>
+  <xacro:property name="center_axle_z" value="0.33"/>
   <!-- Above ground footprint -->
-  <xacro:property name="rear_axle_x" value="${-base_link_x}"/>
-  <!-- Relative to base_link -->
-  <xacro:property name="rear_axle_z" value="0.0"/>
-  <!-- Relative to base_link -->
+  <xacro:property name="rear_axle_z" value="0.33"/>
+  <!-- Relative to rear_alxe -->
   <xacro:property name="roof_datum_x" value="1.88985"/>
   <xacro:property name="roof_datum_z" value="1.23242"/>
+  <!-- Relative to vehicle_bonnet -->
   <xacro:property name="front_bumper_x" value="0.915"/>
-  <!-- Relative to vehicle_bonnet -->
-  <xacro:property name="front_bumper_z" value="${0.23 - (vehicle_bonnet_z + base_link_z)}"/>
+  <xacro:property name="front_bumper_z" value="${0.23 - (vehicle_bonnet_z + center_axle_z)}"/>
   <!-- FOOTPRINT (Delimited by chassis extremes) -->
   <xacro:property name="footprint_front_x" value="3.805"/>

File: av_lxo_description/urdf/mondeo_dca/mondeo_dca_structure.xacro (robot description, xacro)
@@ -2,5 +2,5 @@
 <robot xmlns:xacro="http://www.ros.org/wiki/xacro" name="dbw_mkz">
   <link name="base_footprint"/>
-  <link name="base_link">
+  <link name="center_axle">
     <inertial>
       <origin xyz="0 0 ${centre_grav_z}" rpy="0 0 0"/>
@@ -16,5 +16,5 @@
     </inertial>
     <visual name="chassis">
-      <origin xyz="${1.361 - base_link_x} 0 -0.33647" rpy="0 0 ${pi/2}"/>
+      <origin xyz="${1.361 - center_axle_x} 0 -0.33647" rpy="0 0 ${pi/2}"/>
       <geometry>
         <mesh filename="package://av_lxo_meshes/meshes/mondeo_grey.dae" scale="1 1 1"/>
@@ -23,5 +23,5 @@
     </visual>
     <collision name="chassis_collision">
-      <origin xyz="${1.4621 - base_link_x} -0.03046 0.350609" rpy="${pi/2} 0 -${pi}"/>
+      <origin xyz="${1.4621 - center_axle_x} -0.03046 0.350609" rpy="${pi/2} 0 -${pi}"/>
       <geometry>
         <mesh filename="package://av_lxo_meshes/meshes/body_collision.stl" scale="0.001 0.001 0.001"/>
@@ -31,5 +31,5 @@
   <joint name="${vehicle_bonnet}_joint" type="fixed">
     <origin xyz="${vehicle_bonnet_x} 0 ${vehicle_bonnet_z}" rpy="0 0 0"/>
-    <parent link="base_link"/>
+    <parent link="rear_axle"/>
     <child link="${vehicle_bonnet}"/>
   </joint>
@@ -41,8 +41,8 @@
     </inertial>
   </link>
-  <joint name="rear_axle_joint" type="fixed">
-    <origin xyz="${rear_axle_x} 0 ${rear_axle_z}" rpy="0 0 0"/>
-    <parent link="base_link"/>
-    <child link="rear_axle"/>
+  <joint name="center_axle_joint" type="fixed">
+    <origin xyz="${center_axle_x} 0 0" rpy="0 0 0"/>
+    <parent link="rear_axle"/>
+    <child link="center_axle"/>
   </joint>
   <link name="rear_axle">
@@ -220,6 +220,6 @@
   </link>
   <joint name="front_axle_joint" type="fixed">
-    <origin xyz="${front_axle_x} 0 0" rpy="0 0 0"/>
-    <parent link="base_link"/>
+    <origin xyz="${wheelbase} 0 0" rpy="0 0 0"/>
+    <parent link="rear_axle"/>
     <child link="front_axle"/>
   </joint>
@@ -243,12 +243,12 @@
     </inertial>
   </link>
-  <joint name="base_link" type="fixed">
-    <origin xyz="${base_link_x} 0 ${base_link_z}" rpy="0 0 0"/>
+  <joint name="rear_axle_joint" type="fixed">
+    <origin xyz="0 0 ${rear_axle_z}" rpy="0 0 0"/>
     <parent link="base_footprint"/>
-    <child link="base_link"/>
+    <child link="rear_axle"/>
   </joint>
   <joint name="steer_fl" type="revolute">
     <origin xyz="${front_axle_x} ${wheel_front_y} 0" rpy="0 0 0"/>
-    <parent link="base_link"/>
+    <parent link="rear_axle"/>
     <child link="steer_fl"/>
     <axis xyz="0 0 1.0"/>
@@ -257,5 +257,5 @@
   <joint name="steer_fr" type="revolute">
     <origin xyz="${front_axle_x} -${wheel_front_y} 0" rpy="0 0 0"/>
-    <parent link="base_link"/>
+    <parent link="rear_axle"/>
     <child link="steer_fr"/>
     <axis xyz="0 0 1.0"/>
@@ -279,6 +279,6 @@
   </joint>
   <joint name="wheel_rl" type="continuous">
-    <origin xyz="-${front_axle_x} ${wheel_rear_y} 0" rpy="${pi/2} 0 -${pi}"/>
-    <parent link="base_link"/>
+    <origin xyz="0.0 ${wheel_rear_y} 0" rpy="${pi/2} 0 -${pi}"/>
+    <parent link="rear_axle"/>
     <child link="wheel_rl"/>
     <axis xyz="0 0 1.0"/>
@@ -287,6 +287,6 @@
   </joint>
   <joint name="wheel_rr" type="continuous">
-    <origin xyz="-${front_axle_x} -${wheel_rear_y} 0" rpy="${pi/2} 0 -${pi}"/>
-    <parent link="base_link"/>
+    <origin xyz="0.0 -${wheel_rear_y} 0" rpy="${pi/2} 0 -${pi}"/>
+    <parent link="rear_axle"/>
     <child link="wheel_rr"/>
     <axis xyz="0 0 1.0"/>

Commit message: Rename rear_axle to base_link

File: av_lxo_description/urdf/mondeo_dca/mondeo_dca_params.xacro (robot description, xacro)
@@ -10,9 +10,10 @@
   <xacro:property name="centre_grav_z" value="0.0"/>
   <xacro:property name="wheelbase" value="2.85"/>
-  <!-- Relative to rear_axle -->
+  <!-- ** base_link located at rear_axle **-->
+  <!-- Relative to base_link -->
   <xacro:property name="vehicle_bonnet_x" value="${wheelbase}"/>
-  <!-- Relative to rear_axle -->
+  <!-- Relative to base_link -->
   <xacro:property name="vehicle_bonnet_z" value="${0.69 - center_axle_z}"/>
-  <!-- Relative to rear_axle -->
+  <!-- Relative to base_link -->
   <xacro:property name="front_axle_x" value="${wheelbase}"/>
   <xacro:property name="wheel_front_y" value="0.79121"/>
@@ -23,5 +24,5 @@
   <xacro:property name="center_axle_z" value="0.33"/>
   <!-- Above ground footprint -->
-  <xacro:property name="rear_axle_z" value="0.33"/>
+  <xacro:property name="base_link_z" value="0.33"/>
   <!-- Relative to rear_alxe -->
   <xacro:property name="roof_datum_x" value="1.88985"/>
@@ -32,7 +33,7 @@
   <!-- FOOTPRINT (Delimited by chassis extremes) -->
   <xacro:property name="footprint_front_x" value="3.805"/>
-  <!-- Relative to rear_axle -->
+  <!-- Relative to base_link -->
   <xacro:property name="footprint_rear_x" value="-1.1"/>
-  <!-- Relative to rear_axle -->
+  <!-- Relative to base_link -->
   <xacro:property name="footprint_y" value="${2.14 / 2.0}"/>
   <!-- Symmetric about the centreline -->

File: av_lxo_description/urdf/mondeo_dca/mondeo_dca_sensors.xacro (robot description, xacro)
@@ -192,5 +192,5 @@
     <origin xyz="-0.16666 -0.58893 0.24618" rpy="3.141592654 0 -0.645772"/>
   </xacro:radar>
-  <xacro:radar name="radar_bumper_rear_centre_mount" parent="rear_axle">
+  <xacro:radar name="radar_bumper_rear_centre_mount" parent="base_link">
     <origin xyz="-1.04 0 0.16" rpy="0 0 3.141592654"/>
   </xacro:radar>

File: av_lxo_description/urdf/mondeo_dca/mondeo_dca_structure.xacro (robot description, xacro)
@@ -31,5 +31,5 @@
   <joint name="${vehicle_bonnet}_joint" type="fixed">
     <origin xyz="${vehicle_bonnet_x} 0 ${vehicle_bonnet_z}" rpy="0 0 0"/>
-    <parent link="rear_axle"/>
+    <parent link="base_link"/>
     <child link="${vehicle_bonnet}"/>
   </joint>
@@ -43,8 +43,8 @@
   <joint name="center_axle_joint" type="fixed">
     <origin xyz="${center_axle_x} 0 0" rpy="0 0 0"/>
-    <parent link="rear_axle"/>
+    <parent link="base_link"/>
     <child link="center_axle"/>
   </joint>
-  <link name="rear_axle">
+  <link name="base_link">
     <inertial>
       <origin xyz="0 0 0" rpy="0 0 0"/>
@@ -55,5 +55,5 @@
   <joint name="${roof_datum}_joint" type="fixed">
     <origin xyz="${roof_datum_x} 0 ${roof_datum_z}" rpy="0 0 0"/>
-    <parent link="rear_axle"/>
+    <parent link="base_link"/>
     <child link="${roof_datum}"/>
   </joint>
@@ -221,5 +221,5 @@
   <joint name="front_axle_joint" type="fixed">
     <origin xyz="${wheelbase} 0 0" rpy="0 0 0"/>
-    <parent link="rear_axle"/>
+    <parent link="base_link"/>
     <child link="front_axle"/>
   </joint>
@@ -243,12 +243,12 @@
     </inertial>
   </link>
-  <joint name="rear_axle_joint" type="fixed">
-    <origin xyz="0 0 ${rear_axle_z}" rpy="0 0 0"/>
+  <joint name="base_link_joint" type="fixed">
+    <origin xyz="0 0 ${base_link_z}" rpy="0 0 0"/>
     <parent link="base_footprint"/>
-    <child link="rear_axle"/>
+    <child link="base_link"/>
   </joint>
   <joint name="steer_fl" type="revolute">
     <origin xyz="${front_axle_x} ${wheel_front_y} 0" rpy="0 0 0"/>
-    <parent link="rear_axle"/>
+    <parent link="base_link"/>
     <child link="steer_fl"/>
     <axis xyz="0 0 1.0"/>
@@ -257,5 +257,5 @@
   <joint name="steer_fr" type="revolute">
     <origin xyz="${front_axle_x} -${wheel_front_y} 0" rpy="0 0 0"/>
-    <parent link="rear_axle"/>
+    <parent link="base_link"/>
     <child link="steer_fr"/>
     <axis xyz="0 0 1.0"/>
@@ -280,5 +280,5 @@
   <joint name="wheel_rl" type="continuous">
     <origin xyz="0.0 ${wheel_rear_y} 0" rpy="${pi/2} 0 -${pi}"/>
-    <parent link="rear_axle"/>
+    <parent link="base_link"/>
     <child link="wheel_rl"/>
     <axis xyz="0 0 1.0"/>
@@ -288,5 +288,5 @@
   <joint name="wheel_rr" type="continuous">
     <origin xyz="0.0 -${wheel_rear_y} 0" rpy="${pi/2} 0 -${pi}"/>
-    <parent link="rear_axle"/>
+    <parent link="base_link"/>
     <child link="wheel_rr"/>
     <axis xyz="0 0 1.0"/>
@@ -297,5 +297,5 @@
   <joint name="footprint_fl_joint" type="fixed">
     <origin xyz="${footprint_front_x} ${footprint_y} 0" rpy="0 0 0"/>
-    <parent link="rear_axle"/>
+    <parent link="base_link"/>
     <child link="footprint_fl"/>
   </joint>
@@ -303,5 +303,5 @@
   <joint name="footprint_fr_joint" type="fixed">
     <origin xyz="${footprint_front_x} ${-footprint_y} 0" rpy="0 0 0"/>
-    <parent link="rear_axle"/>
+    <parent link="base_link"/>
     <child link="footprint_fr"/>
   </joint>
@@ -309,5 +309,5 @@
   <joint name="footprint_rl_joint" type="fixed">
     <origin xyz="${footprint_rear_x} ${footprint_y} 0" rpy="0 0 0"/>
-    <parent link="rear_axle"/>
+    <parent link="base_link"/>
     <child link="footprint_rl"/>
   </joint>
@@ -315,5 +315,5 @@
   <joint name="footprint_rr_joint" type="fixed">
     <origin xyz="${footprint_rear_x} ${-footprint_y} 0" rpy="0 0 0"/>
-    <parent link="rear_axle"/>
+    <parent link="base_link"/>
     <child link="footprint_rr"/>
   </joint>
