Commit message: Add camera TF frames derived from mounting frames

File: av_car_description/urdf/mondeo_dca/mondeo_dca_sensors.xacro (robot description, xacro)
@@ -11,48 +11,96 @@
     <origin xyz="-0.11015 0.3 -0.06242" rpy="0 0.087266 0"/>
   </xacro:camera_mount>
+  <xacro:camera_mount name="fsp_l" parent="camera_fsp_l_mount">
+    <origin xyz="0 0 0" rpy="1.5708 3.141592654 1.5708"/>
+  </xacro:camera_mount>
   <xacro:camera_mount name="camera_fsp_r_mount" parent="${roof_datum}">
     <origin xyz="-0.11015 -0.3 -0.06242" rpy="0 0.087266 0"/>
   </xacro:camera_mount>
-  <xacro:camera_mount name="camera_rsspf_l_mount" parent="${roof_datum}">
+  <xacro:camera_mount name="fsp_r" parent="camera_fsp_r_mount">
+    <origin xyz="0 0 0" rpy="1.5708 3.141592654 1.5708"/>
+  </xacro:camera_mount>
+  <xacro:camera_mount name="camera_rspf_l_mount" parent="${roof_datum}">
     <origin xyz="-0.69015 -0.45 -0.00242" rpy="0 0.087266 -1.151917"/>
   </xacro:camera_mount>
-  <xacro:camera_mount name="camera_rsspf_r_mount" parent="${roof_datum}">
+  <xacro:camera_mount name="rspf_l" parent="camera_rspf_l_mount">
+    <origin xyz="0 0 0" rpy="1.5708 3.141592654 1.5708"/>
+  </xacro:camera_mount>
+  <xacro:camera_mount name="camera_rspf_r_mount" parent="${roof_datum}">
     <origin xyz="-0.781503 -0.490673 -0.00242" rpy="0 0.087266 -1.151917"/>
   </xacro:camera_mount>
-  <xacro:camera_mount name="camera_rsspr_l_mount" parent="${roof_datum}">
+  <xacro:camera_mount name="rspf_r" parent="camera_rspf_r_mount">
+    <origin xyz="0 0 0" rpy="1.5708 3.141592654 1.5708"/>
+  </xacro:camera_mount>
+  <xacro:camera_mount name="camera_rspr_l_mount" parent="${roof_datum}">
     <origin xyz="-0.97015 -0.490673 -0.00242" rpy="0 0.087266 -1.989675"/>
   </xacro:camera_mount>
-  <xacro:camera_mount name="camera_rsspr_r_mount" parent="${roof_datum}">
+  <xacro:camera_mount name="rspr_l" parent="camera_rspr_l_mount">
+    <origin xyz="0 0 0" rpy="1.5708 3.141592654 1.5708"/>
+  </xacro:camera_mount>
+  <xacro:camera_mount name="camera_rspr_r_mount" parent="${roof_datum}">
     <origin xyz="-1.061503 -0.450 0.00242" rpy="0 0.087266 -1.989675"/>
+  </xacro:camera_mount>
+  <xacro:camera_mount name="rspr_r" parent="camera_rspr_r_mount">
+    <origin xyz="0 0 0" rpy="1.5708 3.141592654 1.5708"/>
   </xacro:camera_mount>
   <xacro:camera_mount name="camera_rsp_l_mount" parent="${roof_datum}">
     <origin xyz="-1.11015 -0.3 0.00242" rpy="0 0.087266 3.141592654"/>
   </xacro:camera_mount>
+  <xacro:camera_mount name="rsp_l" parent="camera_rsp_l_mount">
+    <origin xyz="0 0 0" rpy="1.5708 0 1.5708"/>
+  </xacro:camera_mount>
   <xacro:camera_mount name="camera_rsp_r_mount" parent="${roof_datum}">
     <origin xyz="-1.11015 0.3 0.00242" rpy="0 0.087266 3.141592654"/>
   </xacro:camera_mount>
-  <xacro:camera_mount name="camera_lsspr_l_mount" parent="${roof_datum}">
+  <xacro:camera_mount name="rsp_r" parent="camera_rsp_r_mount">
+    <origin xyz="0 0 0" rpy="1.5708 3.141592654 1.5708"/>
+  </xacro:camera_mount>
+  <xacro:camera_mount name="camera_lspr_l_mount" parent="${roof_datum}">
     <origin xyz="-1.061503 0.450 0.00242" rpy="0 0.087266 1.989675"/>
   </xacro:camera_mount>
-  <xacro:camera_mount name="camera_lsspr_r_mount" parent="${roof_datum}">
+  <xacro:camera_mount name="lspr_l" parent="camera_lspr_l_mount">
+    <origin xyz="0 0 0" rpy="1.5708 0 1.5708"/>
+  </xacro:camera_mount>
+  <xacro:camera_mount name="camera_lspr_r_mount" parent="${roof_datum}">
     <origin xyz="-0.97015 0.490673 -0.00242" rpy="0 0.087266 1.989675"/>
   </xacro:camera_mount>
-  <xacro:camera_mount name="camera_lsspf_l_mount" parent="${roof_datum}">
+  <xacro:camera_mount name="lspr_r" parent="camera_lspr_r_mount">
+    <origin xyz="0 0 0" rpy="1.5708 0 1.5708"/>
+  </xacro:camera_mount>
+  <xacro:camera_mount name="camera_lspf_l_mount" parent="${roof_datum}">
     <origin xyz="-0.781503 0.490673 -0.00242" rpy="0 0.087266 1.151917"/>
   </xacro:camera_mount>
-  <xacro:camera_mount name="camera_lsspf_r_mount" parent="${roof_datum}">
+  <xacro:camera_mount name="lspf_l" parent="camera_lspf_l_mount">
+    <origin xyz="0 0 0" rpy="1.5708 0 1.5708"/>
+  </xacro:camera_mount>
+  <xacro:camera_mount name="camera_lspf_r_mount" parent="${roof_datum}">
     <origin xyz="-0.69015 0.45 -0.00242" rpy="0 0.087266 1.151917"/>
+  </xacro:camera_mount>
+  <xacro:camera_mount name="lspf_r" parent="camera_lspf_r_mount">
+    <origin xyz="0 0 0" rpy="1.5708 0 1.5708"/>
   </xacro:camera_mount>
   <xacro:camera_mount name="camera_tele1_mount" parent="${roof_datum}">
     <origin xyz="-0.11015 -0.120 -0.06242" rpy="0 0 0"/>
   </xacro:camera_mount>
+  <xacro:camera_mount name="tele1" parent="camera_tele1_mount">
+    <origin xyz="0 0 0" rpy="1.5708 0 1.5708"/>
+  </xacro:camera_mount>
   <xacro:camera_mount name="camera_tele2_mount" parent="${roof_datum}">
     <origin xyz="-0.11015 -0.205 -0.06242" rpy="0 0 0"/>
+  </xacro:camera_mount>
+  <xacro:camera_mount name="tele2" parent="camera_tele2_mount">
+    <origin xyz="0 0 0" rpy="1.5708 0 1.5708"/>
   </xacro:camera_mount>
   <xacro:camera_mount name="camera_ir1_mount" parent="${roof_datum}">
     <origin xyz="-0.11015 0.120 -0.06242" rpy="0 0 0"/>
   </xacro:camera_mount>
+  <xacro:camera_mount name="ir1" parent="camera_ir1_mount">
+    <origin xyz="0 0 0" rpy="1.5708 0 1.5708"/>
+  </xacro:camera_mount>
   <xacro:camera_mount name="camera_ir2_mount" parent="${roof_datum}">
     <origin xyz="-0.11015 0.205 -0.06242" rpy="0 0 0"/>
+  </xacro:camera_mount>
+  <xacro:camera_mount name="ir2" parent="camera_ir2_mount">
+    <origin xyz="0 0 0" rpy="1.5708 0 1.5708"/>
   </xacro:camera_mount>
   <!-- IMU -->

Commit message: WIP: Update camera sensor frame id

File: av_car_description/urdf/mondeo_dca/mondeo_dca_sensors.xacro (robot description, xacro)
@@ -77,5 +77,8 @@
     <origin xyz="-0.69015 0.45 -0.00242" rpy="0 0.087266 1.151917"/>
   </xacro:camera_mount>
-  <xacro:camera_mount name="lspf_r" parent="camera_lspf_r_mount">
+  <xacro:camera_mount name="lspf_r_sensor" parent="camera_lspf_r_mount">
+    <origin xyz="0 0 0" rpy="3.1415 0 0"/>
+  </xacro:camera_mount>
+  <xacro:camera_mount name="lspf_r_optical" parent="lspf_r_sensor">
     <origin xyz="0 0 0" rpy="1.5708 0 1.5708"/>
   </xacro:camera_mount>

Commit message: Add sensor and optical frames for all cameras
 - Sensor frame is a rotation of mount but in camera coordinates
 - Optical frame TF values now 0s will change in future when sensors are
 calibrated with each other (i.e. cross-sensor registration)

File: av_car_description/urdf/mondeo_dca/mondeo_dca_sensors.xacro (robot description, xacro)
@@ -11,66 +11,99 @@
     <origin xyz="-0.11015 0.3 -0.06242" rpy="0 0.087266 0"/>
   </xacro:camera_mount>
-  <xacro:camera_mount name="fsp_l" parent="camera_fsp_l_mount">
-    <origin xyz="0 0 0" rpy="1.5708 3.141592654 1.5708"/>
+  <xacro:camera_mount name="fsp_l_sensor" parent="camera_fsp_l_mount">
+    <origin xyz="0 0 0" rpy="1.5708 3.1415 1.5708"/>
+  </xacro:camera_mount>
+  <xacro:camera_mount name="fsp_l_optical" parent="fsp_l_sensor">
+    <origin xyz="0 0 0" rpy="0 0 0"/>
   </xacro:camera_mount>
   <xacro:camera_mount name="camera_fsp_r_mount" parent="${roof_datum}">
     <origin xyz="-0.11015 -0.3 -0.06242" rpy="0 0.087266 0"/>
   </xacro:camera_mount>
-  <xacro:camera_mount name="fsp_r" parent="camera_fsp_r_mount">
-    <origin xyz="0 0 0" rpy="1.5708 3.141592654 1.5708"/>
+  <xacro:camera_mount name="fsp_r_sensor" parent="camera_fsp_r_mount">
+    <origin xyz="0 0 0" rpy="1.5708 3.1415 1.5708"/>
+  </xacro:camera_mount>
+  <xacro:camera_mount name="fsp_r_optical" parent="fsp_r_sensor">
+    <origin xyz="0 0 0" rpy="0 0 0"/>
   </xacro:camera_mount>
   <xacro:camera_mount name="camera_rspf_l_mount" parent="${roof_datum}">
     <origin xyz="-0.69015 -0.45 -0.00242" rpy="0 0.087266 -1.151917"/>
   </xacro:camera_mount>
-  <xacro:camera_mount name="rspf_l" parent="camera_rspf_l_mount">
-    <origin xyz="0 0 0" rpy="1.5708 3.141592654 1.5708"/>
+  <xacro:camera_mount name="rspf_l_sensor" parent="camera_rspf_l_mount">
+    <origin xyz="0 0 0" rpy="1.5708 3.1415 1.5708"/>
+  </xacro:camera_mount>
+  <xacro:camera_mount name="rspf_l_optical" parent="rspf_l_sensor">
+    <origin xyz="0 0 0" rpy="0 0 0"/>
   </xacro:camera_mount>
   <xacro:camera_mount name="camera_rspf_r_mount" parent="${roof_datum}">
     <origin xyz="-0.781503 -0.490673 -0.00242" rpy="0 0.087266 -1.151917"/>
   </xacro:camera_mount>
-  <xacro:camera_mount name="rspf_r" parent="camera_rspf_r_mount">
-    <origin xyz="0 0 0" rpy="1.5708 3.141592654 1.5708"/>
+  <xacro:camera_mount name="rspf_r_sensor" parent="camera_rspf_r_mount">
+    <origin xyz="0 0 0" rpy="1.5708 3.1415 1.5708"/>
+  </xacro:camera_mount>
+  <xacro:camera_mount name="rspf_r_optical" parent="rspf_r_sensor">
+    <origin xyz="0 0 0" rpy="0 0 0"/>
   </xacro:camera_mount>
   <xacro:camera_mount name="camera_rspr_l_mount" parent="${roof_datum}">
     <origin xyz="-0.97015 -0.490673 -0.00242" rpy="0 0.087266 -1.989675"/>
   </xacro:camera_mount>
-  <xacro:camera_mount name="rspr_l" parent="camera_rspr_l_mount">
-    <origin xyz="0 0 0" rpy="1.5708 3.141592654 1.5708"/>
+  <xacro:camera_mount name="rspr_l_sensor" parent="camera_rspr_l_mount">
+    <origin xyz="0 0 0" rpy="1.5708 3.1415 1.5708"/>
+  </xacro:camera_mount>
+  <xacro:camera_mount name="rspr_l_optical" parent="rspr_l_sensor">
+    <origin xyz="0 0 0" rpy="0 0 0"/>
   </xacro:camera_mount>
   <xacro:camera_mount name="camera_rspr_r_mount" parent="${roof_datum}">
     <origin xyz="-1.061503 -0.450 0.00242" rpy="0 0.087266 -1.989675"/>
   </xacro:camera_mount>
-  <xacro:camera_mount name="rspr_r" parent="camera_rspr_r_mount">
-    <origin xyz="0 0 0" rpy="1.5708 3.141592654 1.5708"/>
+  <xacro:camera_mount name="rspr_r_sensor" parent="camera_rspr_r_mount">
+    <origin xyz="0 0 0" rpy="1.5708 3.1415 1.5708"/>
+  </xacro:camera_mount>
+  <xacro:camera_mount name="rspr_r_optical" parent="rspr_r_sensor">
+    <origin xyz="0 0 0" rpy="0 0 0"/>
   </xacro:camera_mount>
   <xacro:camera_mount name="camera_rsp_l_mount" parent="${roof_datum}">
     <origin xyz="-1.11015 -0.3 0.00242" rpy="0 0.087266 3.141592654"/>
   </xacro:camera_mount>
-  <xacro:camera_mount name="rsp_l" parent="camera_rsp_l_mount">
-    <origin xyz="0 0 0" rpy="1.5708 0 1.5708"/>
+  <xacro:camera_mount name="rsp_l_sensor" parent="camera_rsp_l_mount">
+    <origin xyz="0 0 0" rpy="1.5708 3.1415 1.5708"/>
+  </xacro:camera_mount>
+  <xacro:camera_mount name="rsp_l_optical" parent="rsp_l_sensor">
+    <origin xyz="0 0 0" rpy="0 0 0"/>
   </xacro:camera_mount>
   <xacro:camera_mount name="camera_rsp_r_mount" parent="${roof_datum}">
     <origin xyz="-1.11015 0.3 0.00242" rpy="0 0.087266 3.141592654"/>
   </xacro:camera_mount>
-  <xacro:camera_mount name="rsp_r" parent="camera_rsp_r_mount">
-    <origin xyz="0 0 0" rpy="1.5708 3.141592654 1.5708"/>
+  <xacro:camera_mount name="rsp_r_sensor" parent="camera_rsp_r_mount">
+    <origin xyz="0 0 0" rpy="1.5708 3.1415 1.5708"/>
+  </xacro:camera_mount>
+  <xacro:camera_mount name="rsp_r_optical" parent="rsp_r_sensor">
+    <origin xyz="0 0 0" rpy="0 0 0"/>
   </xacro:camera_mount>
   <xacro:camera_mount name="camera_lspr_l_mount" parent="${roof_datum}">
     <origin xyz="-1.061503 0.450 0.00242" rpy="0 0.087266 1.989675"/>
   </xacro:camera_mount>
-  <xacro:camera_mount name="lspr_l" parent="camera_lspr_l_mount">
-    <origin xyz="0 0 0" rpy="1.5708 0 1.5708"/>
+  <xacro:camera_mount name="lspr_l_sensor" parent="camera_lspr_l_mount">
+    <origin xyz="0 0 0" rpy="1.5708 3.1415 1.5708"/>
+  </xacro:camera_mount>
+  <xacro:camera_mount name="lspr_l_optical" parent="lspr_l_sensor">
+    <origin xyz="0 0 0" rpy="0 0 0"/>
   </xacro:camera_mount>
   <xacro:camera_mount name="camera_lspr_r_mount" parent="${roof_datum}">
     <origin xyz="-0.97015 0.490673 -0.00242" rpy="0 0.087266 1.989675"/>
   </xacro:camera_mount>
-  <xacro:camera_mount name="lspr_r" parent="camera_lspr_r_mount">
-    <origin xyz="0 0 0" rpy="1.5708 0 1.5708"/>
+  <xacro:camera_mount name="lspr_r_sensor" parent="camera_lspr_r_mount">
+    <origin xyz="0 0 0" rpy="1.5708 3.1415 1.5708"/>
+  </xacro:camera_mount>
+  <xacro:camera_mount name="lspr_r_optical" parent="lspr_r_sensor">
+    <origin xyz="0 0 0" rpy="0 0 0"/>
   </xacro:camera_mount>
   <xacro:camera_mount name="camera_lspf_l_mount" parent="${roof_datum}">
     <origin xyz="-0.781503 0.490673 -0.00242" rpy="0 0.087266 1.151917"/>
   </xacro:camera_mount>
-  <xacro:camera_mount name="lspf_l" parent="camera_lspf_l_mount">
-    <origin xyz="0 0 0" rpy="1.5708 0 1.5708"/>
+  <xacro:camera_mount name="lspf_l_sensor" parent="camera_lspf_l_mount">
+    <origin xyz="0 0 0" rpy="1.5708 3.1415 1.5708"/>
+  </xacro:camera_mount>
+  <xacro:camera_mount name="lspf_l_optical" parent="lspf_l_sensor">
+    <origin xyz="0 0 0" rpy="0 0 0"/>
   </xacro:camera_mount>
   <xacro:camera_mount name="camera_lspf_r_mount" parent="${roof_datum}">
@@ -78,32 +111,20 @@
   </xacro:camera_mount>
   <xacro:camera_mount name="lspf_r_sensor" parent="camera_lspf_r_mount">
-    <origin xyz="0 0 0" rpy="3.1415 0 0"/>
+    <origin xyz="0 0 0" rpy="1.5708 3.1415 1.5708"/>
   </xacro:camera_mount>
   <xacro:camera_mount name="lspf_r_optical" parent="lspf_r_sensor">
-    <origin xyz="0 0 0" rpy="1.5708 0 1.5708"/>
+    <origin xyz="0 0 0" rpy="0 0 0"/>
   </xacro:camera_mount>
   <xacro:camera_mount name="camera_tele1_mount" parent="${roof_datum}">
     <origin xyz="-0.11015 -0.120 -0.06242" rpy="0 0 0"/>
   </xacro:camera_mount>
-  <xacro:camera_mount name="tele1" parent="camera_tele1_mount">
-    <origin xyz="0 0 0" rpy="1.5708 0 1.5708"/>
-  </xacro:camera_mount>
   <xacro:camera_mount name="camera_tele2_mount" parent="${roof_datum}">
     <origin xyz="-0.11015 -0.205 -0.06242" rpy="0 0 0"/>
-  </xacro:camera_mount>
-  <xacro:camera_mount name="tele2" parent="camera_tele2_mount">
-    <origin xyz="0 0 0" rpy="1.5708 0 1.5708"/>
   </xacro:camera_mount>
   <xacro:camera_mount name="camera_ir1_mount" parent="${roof_datum}">
     <origin xyz="-0.11015 0.120 -0.06242" rpy="0 0 0"/>
   </xacro:camera_mount>
-  <xacro:camera_mount name="ir1" parent="camera_ir1_mount">
-    <origin xyz="0 0 0" rpy="1.5708 0 1.5708"/>
-  </xacro:camera_mount>
   <xacro:camera_mount name="camera_ir2_mount" parent="${roof_datum}">
     <origin xyz="-0.11015 0.205 -0.06242" rpy="0 0 0"/>
-  </xacro:camera_mount>
-  <xacro:camera_mount name="ir2" parent="camera_ir2_mount">
-    <origin xyz="0 0 0" rpy="1.5708 0 1.5708"/>
   </xacro:camera_mount>
   <!-- IMU -->

Commit message: Add sensor and optical frames for all cameras (#10)
- Sensor frame (in camera z-forwards convention): No translation, only
rotation for camera frame convention
- Optical frame (used by consumers of camera topics): No translation/No
rotation from sensor frame, to be populated by extrinsic calibration.

---------

Co-authored-by: hect95 <hector_cruz95@live.com>

File: av_car_description/urdf/mondeo_dca/mondeo_dca_sensors.xacro (robot description, xacro)
@@ -11,36 +11,108 @@
     <origin xyz="-0.11015 0.3 -0.06242" rpy="0 0.087266 0"/>
   </xacro:camera_mount>
+  <xacro:camera_mount name="camera_fsp_l_sensor" parent="camera_fsp_l_mount">
+    <origin xyz="0 0 0" rpy="1.5708 3.1415 1.5708"/>
+  </xacro:camera_mount>
+  <xacro:camera_mount name="camera_fsp_l_optical" parent="camera_fsp_l_sensor">
+    <origin xyz="0 0 0" rpy="0 0 0"/>
+  </xacro:camera_mount>
   <xacro:camera_mount name="camera_fsp_r_mount" parent="${roof_datum}">
     <origin xyz="-0.11015 -0.3 -0.06242" rpy="0 0.087266 0"/>
   </xacro:camera_mount>
-  <xacro:camera_mount name="camera_rsspf_l_mount" parent="${roof_datum}">
+  <xacro:camera_mount name="camera_fsp_r_sensor" parent="camera_fsp_r_mount">
+    <origin xyz="0 0 0" rpy="1.5708 3.1415 1.5708"/>
+  </xacro:camera_mount>
+  <xacro:camera_mount name="camera_fsp_r_optical" parent="camera_fsp_r_sensor">
+    <origin xyz="0 0 0" rpy="0 0 0"/>
+  </xacro:camera_mount>
+  <xacro:camera_mount name="camera_rspf_l_mount" parent="${roof_datum}">
     <origin xyz="-0.69015 -0.45 -0.00242" rpy="0 0.087266 -1.151917"/>
   </xacro:camera_mount>
-  <xacro:camera_mount name="camera_rsspf_r_mount" parent="${roof_datum}">
+  <xacro:camera_mount name="camera_rspf_l_sensor" parent="camera_rspf_l_mount">
+    <origin xyz="0 0 0" rpy="1.5708 3.1415 1.5708"/>
+  </xacro:camera_mount>
+  <xacro:camera_mount name="camera_rspf_l_optical" parent="camera_rspf_l_sensor">
+    <origin xyz="0 0 0" rpy="0 0 0"/>
+  </xacro:camera_mount>
+  <xacro:camera_mount name="camera_rspf_r_mount" parent="${roof_datum}">
     <origin xyz="-0.781503 -0.490673 -0.00242" rpy="0 0.087266 -1.151917"/>
   </xacro:camera_mount>
-  <xacro:camera_mount name="camera_rsspr_l_mount" parent="${roof_datum}">
+  <xacro:camera_mount name="camera_rspf_r_sensor" parent="camera_rspf_r_mount">
+    <origin xyz="0 0 0" rpy="1.5708 3.1415 1.5708"/>
+  </xacro:camera_mount>
+  <xacro:camera_mount name="camera_rspf_r_optical" parent="camera_rspf_r_sensor">
+    <origin xyz="0 0 0" rpy="0 0 0"/>
+  </xacro:camera_mount>
+  <xacro:camera_mount name="camera_rspr_l_mount" parent="${roof_datum}">
     <origin xyz="-0.97015 -0.490673 -0.00242" rpy="0 0.087266 -1.989675"/>
   </xacro:camera_mount>
-  <xacro:camera_mount name="camera_rsspr_r_mount" parent="${roof_datum}">
+  <xacro:camera_mount name="camera_rspr_l_sensor" parent="camera_rspr_l_mount">
+    <origin xyz="0 0 0" rpy="1.5708 3.1415 1.5708"/>
+  </xacro:camera_mount>
+  <xacro:camera_mount name="camera_rspr_l_optical" parent="camera_rspr_l_sensor">
+    <origin xyz="0 0 0" rpy="0 0 0"/>
+  </xacro:camera_mount>
+  <xacro:camera_mount name="camera_rspr_r_mount" parent="${roof_datum}">
     <origin xyz="-1.061503 -0.450 0.00242" rpy="0 0.087266 -1.989675"/>
+  </xacro:camera_mount>
+  <xacro:camera_mount name="camera_rspr_r_sensor" parent="camera_rspr_r_mount">
+    <origin xyz="0 0 0" rpy="1.5708 3.1415 1.5708"/>
+  </xacro:camera_mount>
+  <xacro:camera_mount name="camera_rspr_r_optical" parent="camera_rspr_r_sensor">
+    <origin xyz="0 0 0" rpy="0 0 0"/>
   </xacro:camera_mount>
   <xacro:camera_mount name="camera_rsp_l_mount" parent="${roof_datum}">
     <origin xyz="-1.11015 -0.3 0.00242" rpy="0 0.087266 3.141592654"/>
   </xacro:camera_mount>
+  <xacro:camera_mount name="camera_rsp_l_sensor" parent="camera_rsp_l_mount">
+    <origin xyz="0 0 0" rpy="1.5708 3.1415 1.5708"/>
+  </xacro:camera_mount>
+  <xacro:camera_mount name="camera_rsp_l_optical" parent="camera_rsp_l_sensor">
+    <origin xyz="0 0 0" rpy="0 0 0"/>
+  </xacro:camera_mount>
   <xacro:camera_mount name="camera_rsp_r_mount" parent="${roof_datum}">
     <origin xyz="-1.11015 0.3 0.00242" rpy="0 0.087266 3.141592654"/>
   </xacro:camera_mount>
-  <xacro:camera_mount name="camera_lsspr_l_mount" parent="${roof_datum}">
+  <xacro:camera_mount name="camera_rsp_r_sensor" parent="camera_rsp_r_mount">
+    <origin xyz="0 0 0" rpy="1.5708 3.1415 1.5708"/>
+  </xacro:camera_mount>
+  <xacro:camera_mount name="camera_rsp_r_optical" parent="camera_rsp_r_sensor">
+    <origin xyz="0 0 0" rpy="0 0 0"/>
+  </xacro:camera_mount>
+  <xacro:camera_mount name="camera_lspr_l_mount" parent="${roof_datum}">
     <origin xyz="-1.061503 0.450 0.00242" rpy="0 0.087266 1.989675"/>
   </xacro:camera_mount>
-  <xacro:camera_mount name="camera_lsspr_r_mount" parent="${roof_datum}">
+  <xacro:camera_mount name="camera_lspr_l_sensor" parent="camera_lspr_l_mount">
+    <origin xyz="0 0 0" rpy="1.5708 3.1415 1.5708"/>
+  </xacro:camera_mount>
+  <xacro:camera_mount name="camera_lspr_l_optical" parent="camera_lspr_l_sensor">
+    <origin xyz="0 0 0" rpy="0 0 0"/>
+  </xacro:camera_mount>
+  <xacro:camera_mount name="camera_lspr_r_mount" parent="${roof_datum}">
     <origin xyz="-0.97015 0.490673 -0.00242" rpy="0 0.087266 1.989675"/>
   </xacro:camera_mount>
-  <xacro:camera_mount name="camera_lsspf_l_mount" parent="${roof_datum}">
+  <xacro:camera_mount name="camera_lspr_r_sensor" parent="camera_lspr_r_mount">
+    <origin xyz="0 0 0" rpy="1.5708 3.1415 1.5708"/>
+  </xacro:camera_mount>
+  <xacro:camera_mount name="camera_lspr_r_optical" parent="camera_lspr_r_sensor">
+    <origin xyz="0 0 0" rpy="0 0 0"/>
+  </xacro:camera_mount>
+  <xacro:camera_mount name="camera_lspf_l_mount" parent="${roof_datum}">
     <origin xyz="-0.781503 0.490673 -0.00242" rpy="0 0.087266 1.151917"/>
   </xacro:camera_mount>
-  <xacro:camera_mount name="camera_lsspf_r_mount" parent="${roof_datum}">
+  <xacro:camera_mount name="camera_lspf_l_sensor" parent="camera_lspf_l_mount">
+    <origin xyz="0 0 0" rpy="1.5708 3.1415 1.5708"/>
+  </xacro:camera_mount>
+  <xacro:camera_mount name="camera_lspf_l_optical" parent="camera_lspf_l_sensor">
+    <origin xyz="0 0 0" rpy="0 0 0"/>
+  </xacro:camera_mount>
+  <xacro:camera_mount name="camera_lspf_r_mount" parent="${roof_datum}">
     <origin xyz="-0.69015 0.45 -0.00242" rpy="0 0.087266 1.151917"/>
+  </xacro:camera_mount>
+  <xacro:camera_mount name="camera_lspf_r_sensor" parent="camera_lspf_r_mount">
+    <origin xyz="0 0 0" rpy="1.5708 3.1415 1.5708"/>
+  </xacro:camera_mount>
+  <xacro:camera_mount name="camera_lspf_r_optical" parent="camera_lspf_r_sensor">
+    <origin xyz="0 0 0" rpy="0 0 0"/>
   </xacro:camera_mount>
   <xacro:camera_mount name="camera_tele1_mount" parent="${roof_datum}">
