Commit message: Add calibrated camera extrinsics

File: av_car_description/urdf/mondeo_dca/mondeo_dca_sensors.xacro (robot description, xacro)
@@ -15,5 +15,5 @@
   </xacro:camera_mount>
   <xacro:camera_mount name="camera_fsp_l_optical" parent="camera_fsp_l_sensor">
-    <origin xyz="0 0 0" rpy="0 0 0"/>
+    <origin xyz="-0.00574471 -0.0386351 0.143683" rpy="0.0450218 0.00437583 -0.00877551" />
   </xacro:camera_mount>
   <xacro:camera_mount name="camera_fsp_r_mount" parent="${roof_datum}">
@@ -33,5 +33,5 @@
   </xacro:camera_mount>
   <xacro:camera_mount name="camera_rspf_l_optical" parent="camera_rspf_l_sensor">
-    <origin xyz="0 0 0" rpy="0 0 0"/>
+    <origin xyz="-0.028194 -0.0153176 0.0970391" rpy="0.0175874 -0.00675707 0.0342503" />
   </xacro:camera_mount>
   <xacro:camera_mount name="camera_rspf_r_mount" parent="${roof_datum}">
@@ -60,5 +60,5 @@
   </xacro:camera_mount>
   <xacro:camera_mount name="camera_rspr_r_optical" parent="camera_rspr_r_sensor">
-    <origin xyz="0 0 0" rpy="0 0 0"/>
+    <origin xyz="-0.101587 0.0158039 0.0444535" rpy="-0.0104926 0.00151955 0.0329238" />
   </xacro:camera_mount>
   <xacro:camera_mount name="camera_rsp_l_mount" parent="${roof_datum}">
@@ -69,5 +69,5 @@
   </xacro:camera_mount>
   <xacro:camera_mount name="camera_rsp_l_optical" parent="camera_rsp_l_sensor">
-    <origin xyz="0 0 0" rpy="0 0 0"/>
+    <origin xyz="-0.0168454 0.014722 0.114717" rpy="-0.0332488 -0.0086389 0.00423322" />
   </xacro:camera_mount>
   <xacro:camera_mount name="camera_rsp_r_mount" parent="${roof_datum}">
@@ -87,5 +87,5 @@
   </xacro:camera_mount>
   <xacro:camera_mount name="camera_lspr_l_optical" parent="camera_lspr_l_sensor">
-    <origin xyz="0 0 0" rpy="0 0 0"/>
+    <origin xyz="0.0850904 0.0215383 -0.0012268" rpy="-0.00558708 -0.00439865 -0.0242586" />
   </xacro:camera_mount>
   <xacro:camera_mount name="camera_lspr_r_mount" parent="${roof_datum}">
@@ -114,5 +114,5 @@
   </xacro:camera_mount>
   <xacro:camera_mount name="camera_lspf_r_optical" parent="camera_lspf_r_sensor">
-    <origin xyz="0 0 0" rpy="0 0 0"/>
+    <origin xyz="0.00369163 -0.002197 0.0529729" rpy="0.0209065 0.000883984 -0.0273617" />
   </xacro:camera_mount>
   <xacro:camera_mount name="camera_tele1_mount" parent="${roof_datum}">

Commit message: Update cam extrinsics for new roi

File: av_car_description/urdf/mondeo_dca/mondeo_dca_sensors.xacro (robot description, xacro)
@@ -15,5 +15,5 @@
   </xacro:camera_mount>
   <xacro:camera_mount name="camera_fsp_l_optical" parent="camera_fsp_l_sensor">
-    <origin xyz="-0.00574471 -0.0386351 0.143683" rpy="0.0450218 0.00437583 -0.00877551" />
+    <origin xyz="-0.0018577 -0.0458795 0.104066" rpy="0.0337803 0.001314 -0.0119997"/>
   </xacro:camera_mount>
   <xacro:camera_mount name="camera_fsp_r_mount" parent="${roof_datum}">
@@ -33,5 +33,5 @@
   </xacro:camera_mount>
   <xacro:camera_mount name="camera_rspf_l_optical" parent="camera_rspf_l_sensor">
-    <origin xyz="-0.028194 -0.0153176 0.0970391" rpy="0.0175874 -0.00675707 0.0342503" />
+    <origin xyz="-0.0317939 -0.0155957 0.0925816" rpy="0.0169439 -0.00863387 0.0310647"/>
   </xacro:camera_mount>
   <xacro:camera_mount name="camera_rspf_r_mount" parent="${roof_datum}">
@@ -60,5 +60,5 @@
   </xacro:camera_mount>
   <xacro:camera_mount name="camera_rspr_r_optical" parent="camera_rspr_r_sensor">
-    <origin xyz="-0.101587 0.0158039 0.0444535" rpy="-0.0104926 0.00151955 0.0329238" />
+    <origin xyz="-0.112357 -0.00142148 0.0607117" rpy="-0.0166038 0.000711473 0.0351392"/>
   </xacro:camera_mount>
   <xacro:camera_mount name="camera_rsp_l_mount" parent="${roof_datum}">
@@ -69,5 +69,5 @@
   </xacro:camera_mount>
   <xacro:camera_mount name="camera_rsp_l_optical" parent="camera_rsp_l_sensor">
-    <origin xyz="-0.0168454 0.014722 0.114717" rpy="-0.0332488 -0.0086389 0.00423322" />
+    <origin xyz="0.0182792 0.00339082 0.0755967" rpy="-0.0296637 -0.00489342 -0.0013936"/>
   </xacro:camera_mount>
   <xacro:camera_mount name="camera_rsp_r_mount" parent="${roof_datum}">
@@ -87,5 +87,5 @@
   </xacro:camera_mount>
   <xacro:camera_mount name="camera_lspr_l_optical" parent="camera_lspr_l_sensor">
-    <origin xyz="0.0850904 0.0215383 -0.0012268" rpy="-0.00558708 -0.00439865 -0.0242586" />
+    <origin xyz="0.101295 0.0114506 0.025199" rpy="-0.0143108 -0.00899993 -0.0256042"/>
   </xacro:camera_mount>
   <xacro:camera_mount name="camera_lspr_r_mount" parent="${roof_datum}">
@@ -114,5 +114,5 @@
   </xacro:camera_mount>
   <xacro:camera_mount name="camera_lspf_r_optical" parent="camera_lspf_r_sensor">
-    <origin xyz="0.00369163 -0.002197 0.0529729" rpy="0.0209065 0.000883984 -0.0273617" />
+    <origin xyz="-0.00129624 -0.00739873 0.116781" rpy="0.00287316 -0.000663669 -0.0262024"/>
   </xacro:camera_mount>
   <xacro:camera_mount name="camera_tele1_mount" parent="${roof_datum}">

Commit message: New camera extrinsics (#16)
- Update camera extrinsics based on camera lidar calibration
- The extrinsics are based on camera configuration defined in
https://github.com/ipab-rad/av_camera/pull/7

File: av_car_description/urdf/mondeo_dca/mondeo_dca_sensors.xacro (robot description, xacro)
@@ -15,5 +15,5 @@
   </xacro:camera_mount>
   <xacro:camera_mount name="camera_fsp_l_optical" parent="camera_fsp_l_sensor">
-    <origin xyz="0 0 0" rpy="0 0 0"/>
+    <origin xyz="-0.0018577 -0.0458795 0.104066" rpy="0.0337803 0.001314 -0.0119997"/>
   </xacro:camera_mount>
   <xacro:camera_mount name="camera_fsp_r_mount" parent="${roof_datum}">
@@ -33,5 +33,5 @@
   </xacro:camera_mount>
   <xacro:camera_mount name="camera_rspf_l_optical" parent="camera_rspf_l_sensor">
-    <origin xyz="0 0 0" rpy="0 0 0"/>
+    <origin xyz="-0.0317939 -0.0155957 0.0925816" rpy="0.0169439 -0.00863387 0.0310647"/>
   </xacro:camera_mount>
   <xacro:camera_mount name="camera_rspf_r_mount" parent="${roof_datum}">
@@ -60,5 +60,5 @@
   </xacro:camera_mount>
   <xacro:camera_mount name="camera_rspr_r_optical" parent="camera_rspr_r_sensor">
-    <origin xyz="0 0 0" rpy="0 0 0"/>
+    <origin xyz="-0.112357 -0.00142148 0.0607117" rpy="-0.0166038 0.000711473 0.0351392"/>
   </xacro:camera_mount>
   <xacro:camera_mount name="camera_rsp_l_mount" parent="${roof_datum}">
@@ -69,5 +69,5 @@
   </xacro:camera_mount>
   <xacro:camera_mount name="camera_rsp_l_optical" parent="camera_rsp_l_sensor">
-    <origin xyz="0 0 0" rpy="0 0 0"/>
+    <origin xyz="0.0182792 0.00339082 0.0755967" rpy="-0.0296637 -0.00489342 -0.0013936"/>
   </xacro:camera_mount>
   <xacro:camera_mount name="camera_rsp_r_mount" parent="${roof_datum}">
@@ -87,5 +87,5 @@
   </xacro:camera_mount>
   <xacro:camera_mount name="camera_lspr_l_optical" parent="camera_lspr_l_sensor">
-    <origin xyz="0 0 0" rpy="0 0 0"/>
+    <origin xyz="0.101295 0.0114506 0.025199" rpy="-0.0143108 -0.00899993 -0.0256042"/>
   </xacro:camera_mount>
   <xacro:camera_mount name="camera_lspr_r_mount" parent="${roof_datum}">
@@ -114,5 +114,5 @@
   </xacro:camera_mount>
   <xacro:camera_mount name="camera_lspf_r_optical" parent="camera_lspf_r_sensor">
-    <origin xyz="0 0 0" rpy="0 0 0"/>
+    <origin xyz="-0.00129624 -0.00739873 0.116781" rpy="0.00287316 -0.000663669 -0.0262024"/>
   </xacro:camera_mount>
   <xacro:camera_mount name="camera_tele1_mount" parent="${roof_datum}">

Commit message: Update fsp_l camera tf

File: av_car_description/urdf/mondeo_dca/mondeo_dca_sensors.xacro (robot description, xacro)
@@ -15,5 +15,5 @@
   </xacro:camera_mount>
   <xacro:camera_mount name="camera_fsp_l_optical" parent="camera_fsp_l_sensor">
-    <origin xyz="-0.0018577 -0.0458795 0.104066" rpy="0.0337803 0.001314 -0.0119997"/>
+    <origin xyz="-0.0159515 -0.0271456 0.114486" rpy="0.0368413 0.00292173 -0.009337"/>
   </xacro:camera_mount>
   <xacro:camera_mount name="camera_fsp_r_mount" parent="${roof_datum}">

Commit message: WIP: Add calibrated tf for left and right lidars

File: av_car_description/urdf/mondeo_dca/mondeo_dca_sensors.xacro (robot description, xacro)
@@ -150,9 +150,15 @@
     <origin xyz="-0.66015 0 0.19758" rpy="0 0 0"/>
   </xacro:lidar>
-  <xacro:lidar name="lidar_left" parent="${roof_datum}">
+  <xacro:lidar name="lidar_left_old" parent="${roof_datum}">
     <origin xyz="-0.03015 0.720 -0.22242" rpy="-0.087266 0.087266 0.6562438"/>
   </xacro:lidar>
-  <xacro:lidar name="lidar_right" parent="${roof_datum}">
+  <xacro:lidar name="lidar_left" parent="vehicle_roof_datum">
+    <origin xyz="0.0107329 0.728872 -0.116884" rpy="-0.0388081 0.102642 0.65186" />
+  </xacro:lidar>
+  <xacro:lidar name="lidar_right_old" parent="${roof_datum}">
     <origin xyz="-0.03015 -0.720 -0.22242" rpy="0.087266 0.087266 -0.6562438"/>
+  </xacro:lidar>
+  <xacro:lidar name="lidar_right" parent="vehicle_roof_datum">
+    <origin xyz="-0.0115331 -0.705366 -0.133119" rpy="0.026757 0.0875472 -0.655852" />
   </xacro:lidar>
   <xacro:lidar name="lidar_ouster_top" parent="${roof_datum}">

Commit message: WIP: Add lidar extrinsics v2

File: av_car_description/urdf/mondeo_dca/mondeo_dca_sensors.xacro (robot description, xacro)
@@ -150,15 +150,21 @@
     <origin xyz="-0.66015 0 0.19758" rpy="0 0 0"/>
   </xacro:lidar>
-  <xacro:lidar name="lidar_left_old" parent="${roof_datum}">
+  <xacro:lidar name="lidar_left_no_calib" parent="${roof_datum}">
     <origin xyz="-0.03015 0.720 -0.22242" rpy="-0.087266 0.087266 0.6562438"/>
   </xacro:lidar>
-  <xacro:lidar name="lidar_left" parent="vehicle_roof_datum">
+  <xacro:lidar name="lidar_left_calib_v1" parent="vehicle_roof_datum">
     <origin xyz="0.0107329 0.728872 -0.116884" rpy="-0.0388081 0.102642 0.65186" />
   </xacro:lidar>
-  <xacro:lidar name="lidar_right_old" parent="${roof_datum}">
+  <xacro:lidar name="lidar_left" parent="vehicle_roof_datum">
+    <origin xyz="0.0124227 0.727969 -0.112672" rpy="-0.037683 0.102063 0.651836" />
+  </xacro:lidar>
+  <xacro:lidar name="lidar_right_no_calib" parent="${roof_datum}">
     <origin xyz="-0.03015 -0.720 -0.22242" rpy="0.087266 0.087266 -0.6562438"/>
   </xacro:lidar>
+  <xacro:lidar name="lidar_right_calib_v1" parent="vehicle_roof_datum">
+    <origin xyz="-0.0115331 -0.705366 -0.133119" rpy="0.026757 0.0875472 -0.655852" />
+  </xacro:lidar>
   <xacro:lidar name="lidar_right" parent="vehicle_roof_datum">
-    <origin xyz="-0.0115331 -0.705366 -0.133119" rpy="0.026757 0.0875472 -0.655852" />
+    <origin xyz="-0.00715063 -0.714411 -0.160957" rpy="0.0316876 0.0944851 -0.655334" />
   </xacro:lidar>
   <xacro:lidar name="lidar_ouster_top" parent="${roof_datum}">

Commit message: Remove debug lidar frames

File: av_car_description/urdf/mondeo_dca/mondeo_dca_sensors.xacro (robot description, xacro)
@@ -150,21 +150,9 @@
     <origin xyz="-0.66015 0 0.19758" rpy="0 0 0"/>
   </xacro:lidar>
-  <xacro:lidar name="lidar_left_no_calib" parent="${roof_datum}">
-    <origin xyz="-0.03015 0.720 -0.22242" rpy="-0.087266 0.087266 0.6562438"/>
+  <xacro:lidar name="lidar_left" parent="${roof_datum}">
+    <origin xyz="0.0124227 0.727969 -0.112672" rpy="-0.037683 0.102063 0.651836"/>
   </xacro:lidar>
-  <xacro:lidar name="lidar_left_calib_v1" parent="vehicle_roof_datum">
-    <origin xyz="0.0107329 0.728872 -0.116884" rpy="-0.0388081 0.102642 0.65186" />
-  </xacro:lidar>
-  <xacro:lidar name="lidar_left" parent="vehicle_roof_datum">
-    <origin xyz="0.0124227 0.727969 -0.112672" rpy="-0.037683 0.102063 0.651836" />
-  </xacro:lidar>
-  <xacro:lidar name="lidar_right_no_calib" parent="${roof_datum}">
-    <origin xyz="-0.03015 -0.720 -0.22242" rpy="0.087266 0.087266 -0.6562438"/>
-  </xacro:lidar>
-  <xacro:lidar name="lidar_right_calib_v1" parent="vehicle_roof_datum">
-    <origin xyz="-0.0115331 -0.705366 -0.133119" rpy="0.026757 0.0875472 -0.655852" />
-  </xacro:lidar>
-  <xacro:lidar name="lidar_right" parent="vehicle_roof_datum">
-    <origin xyz="-0.00715063 -0.714411 -0.160957" rpy="0.0316876 0.0944851 -0.655334" />
+  <xacro:lidar name="lidar_right" parent="${roof_datum}">
+    <origin xyz="-0.00715063 -0.714411 -0.160957" rpy="0.0316876 0.0944851 -0.655334"/>
   </xacro:lidar>
   <xacro:lidar name="lidar_ouster_top" parent="${roof_datum}">

Commit message: Add lidar_x_mount frames
- Add  lidar mount frames and adjust
  lidar_x_mount -> lidar_x based on calibration
- Mount frames are considered to be the old
  vehicle_roof_datum -> lidar_x TF

File: av_car_description/urdf/mondeo_dca/mondeo_dca_sensors.xacro (robot description, xacro)
@@ -147,12 +147,15 @@
   </xacro:gps>
   <!-- LIDAR -->
-  <xacro:lidar name="lidar_top" parent="${roof_datum}">
-    <origin xyz="-0.66015 0 0.19758" rpy="0 0 0"/>
+  <xacro:lidar name="lidar_left_mount" parent="${roof_datum}">
+    <origin xyz="-0.03015 0.720 -0.22242" rpy="-0.087266 0.087266 0.6562438"/>
   </xacro:lidar>
-  <xacro:lidar name="lidar_left" parent="${roof_datum}">
-    <origin xyz="0.0124227 0.727969 -0.112672" rpy="-0.037683 0.102063 0.651836"/>
+  <xacro:lidar name="lidar_left" parent="lidar_left_mount">
+    <origin xyz="0.0288801 -0.0294088 0.110552" rpy="0.0499763 0.0151241 -0.00307838"/>
   </xacro:lidar>
-  <xacro:lidar name="lidar_right" parent="${roof_datum}">
-    <origin xyz="-0.00715063 -0.714411 -0.160957" rpy="0.0316876 0.0944851 -0.655334"/>
+  <xacro:lidar name="lidar_right_mount" parent="${roof_datum}">
+    <origin xyz="-0.03015 -0.720 -0.22242" rpy="0.087266 0.087266 -0.6562438"/>
+  </xacro:lidar>
+  <xacro:lidar name="lidar_right" parent="lidar_right_mount">
+    <origin xyz="0.00939891 0.0238397 0.0606727" rpy="-0.0556599 0.00727062 0.000273152"/>
   </xacro:lidar>
   <xacro:lidar name="lidar_ouster_top" parent="${roof_datum}">

Commit message: Update lidars extrinsics (#19)
* Refactor LIDAR mounting structure based on LIDAR calibration.
  - Perform adjustments based on calibration between `lidar_ouster_top` and both `lidar_left`
    and `lidar_right`.
    - Update the old chain: `vehicle_roof_datum -> lidar_left` and 
      `vehicle_roof_datum -> lidar_right` to:
      - `vehicle_roof_datum -> lidar_left_mount -> lidar_left`
      - `vehicle_roof_datum -> lidar_right_mount -> lidar_right`
  - Ensure that the new chain `vehicle_roof_datum -> lidar_x_mount` matches 
    the old `vehicle_roof_datum -> lidar_x` TF for future reference.

File: av_car_description/urdf/mondeo_dca/mondeo_dca_sensors.xacro (robot description, xacro)
@@ -147,12 +147,15 @@
   </xacro:gps>
   <!-- LIDAR -->
-  <xacro:lidar name="lidar_top" parent="${roof_datum}">
-    <origin xyz="-0.66015 0 0.19758" rpy="0 0 0"/>
-  </xacro:lidar>
-  <xacro:lidar name="lidar_left" parent="${roof_datum}">
+  <xacro:lidar name="lidar_left_mount" parent="${roof_datum}">
     <origin xyz="-0.03015 0.720 -0.22242" rpy="-0.087266 0.087266 0.6562438"/>
   </xacro:lidar>
-  <xacro:lidar name="lidar_right" parent="${roof_datum}">
+  <xacro:lidar name="lidar_left" parent="lidar_left_mount">
+    <origin xyz="0.0288801 -0.0294088 0.110552" rpy="0.0499763 0.0151241 -0.00307838"/>
+  </xacro:lidar>
+  <xacro:lidar name="lidar_right_mount" parent="${roof_datum}">
     <origin xyz="-0.03015 -0.720 -0.22242" rpy="0.087266 0.087266 -0.6562438"/>
+  </xacro:lidar>
+  <xacro:lidar name="lidar_right" parent="lidar_right_mount">
+    <origin xyz="0.00939891 0.0238397 0.0606727" rpy="-0.0556599 0.00727062 0.000273152"/>
   </xacro:lidar>
   <xacro:lidar name="lidar_ouster_top" parent="${roof_datum}">

Commit message: Fix IMUs and GPS antennas TF (#20)
* Add `*_mount` and `*_sensor` chains for IMUs/GPS
  - Define `imu_rear_mount` -> `imu_rear_sensor` and
  `imu_fps_r_mount` -> `imu_fps_r_sensor` TFs
  - `*_mount` frames describe the physical sensor
  orientation
  - `*_sensor` frames describe the orientation that is
  consistent with the microstrain IMU ROS driver ENU measurements
  - Fix `imu_rear_mount` Y translation based on in-house
  measurements
  - Fix `gps_antenna\_*_mount` translation based on in-house
  measurements
  - Define `gps_antenna\_*_mount` -> `gps_antenna\_*_sensor` TF
    based on GNSS antenna hight relative to mount
* Remove `oxts*` frames and parameters as the sensor is no longer
  mounted in the vehicle

File: av_car_description/urdf/mondeo_dca/mondeo_dca_sensors.xacro (robot description, xacro)
@@ -129,20 +129,28 @@
   </xacro:camera_mount>
   <!-- IMU -->
-  <xacro:imu imu="imu_rear_mount">
-    <origin xyz="${oxts_x-0.19} ${oxts_y+0.23} ${oxts_z-0.44}" rpy="0 0 0"/>
+  <xacro:imu imu="imu_rear_mount" parent="${roof_datum}">
+    <origin xyz="-2.67 0.0 -1.102" rpy="0.0 3.14159 -1.5708"/>
   </xacro:imu>
-  <xacro:imu imu="imu_fsp_r_mount">
-    <origin xyz="-0.23515 -0.355 -0.05442" rpy="0 0 0"/>
+  <xacro:imu imu="imu_rear_sensor" parent="imu_rear_mount">
+    <origin xyz="0.0 0.0 0.0" rpy="3.14159 0.0 0.0 "/>
   </xacro:imu>
-  <!-- OXTS -->
-  <xacro:oxts name="oxts">
-    <origin xyz="${oxts_x} ${oxts_y} ${oxts_z}" rpy="0.0 0.0 0.0"/>
-  </xacro:oxts>
+  <xacro:imu imu="imu_fsp_r_mount" parent="${roof_datum}">
+    <origin xyz="-0.23515 -0.355 -0.05442" rpy="0.0 3.14159 -1.5708"/>
+  </xacro:imu>
+  <xacro:imu imu="imu_fsp_r_sensor" parent="imu_fsp_r_mount">
+    <origin xyz="0.0 0.0 0.0" rpy="3.14159 0.0 0.0"/>
+  </xacro:imu>
   <!-- GPS -->
-  <xacro:gps name="gps_antenna_right_mount">
+  <xacro:gps name="gps_antenna_right_mount" parent="${roof_datum}">
     <origin xyz="${gps_antenna_base_left_x} ${-gps_antenna_base_left_y} ${gps_antenna_base_left_z}" rpy="0 0 0"/>
   </xacro:gps>
-  <xacro:gps name="gps_antenna_left_mount">
+  <xacro:gps name="gps_antenna_right_sensor" parent="gps_antenna_right_mount">
+    <origin xyz="0.0 0.0 ${gps_antenna_sensor_z}" rpy="0 0 0"/>
+  </xacro:gps>
+  <xacro:gps name="gps_antenna_left_mount" parent="${roof_datum}">
     <origin xyz="${gps_antenna_base_left_x} ${gps_antenna_base_left_y} ${gps_antenna_base_left_z}" rpy="0 0 0"/>
+  </xacro:gps>
+  <xacro:gps name="gps_antenna_left_sensor" parent="gps_antenna_left_mount">
+    <origin xyz="0.0 0.0 ${gps_antenna_sensor_z}" rpy="0 0 0"/>
   </xacro:gps>
   <!-- LIDAR -->

Commit message: Add fsp_l calibration tf

File: av_car_description/urdf/mondeo_dca/mondeo_dca_sensors.xacro (robot description, xacro)
@@ -15,5 +15,5 @@
   </xacro:camera_mount>
   <xacro:camera_mount name="camera_fsp_l_optical" parent="camera_fsp_l_sensor">
-    <origin xyz="-0.0159515 -0.0271456 0.114486" rpy="0.0368413 0.00292173 -0.009337"/>
+    <origin xyz="-0.011874 0.049085 0.079928" rpy="0.000929 -0.005284 -0.007228"/>
   </xacro:camera_mount>
   <xacro:camera_mount name="camera_fsp_r_mount" parent="${roof_datum}">
@@ -167,6 +167,6 @@
     <origin xyz="0.00939891 0.0238397 0.0606727" rpy="-0.0556599 0.00727062 0.000273152"/>
   </xacro:lidar>
-  <xacro:lidar name="lidar_ouster_top" parent="${roof_datum}">
-    <origin xyz="-0.65855 0 0.21849" rpy="0 -0.017453 0"/>
+  <xacro:lidar name="lidar_top" parent="${roof_datum}">
+    <origin xyz="-0.65855 0 0.26" rpy="0 0 1.5708"/>
   </xacro:lidar>
   <!-- RADAR -->

Commit message: Update lidar frames
- Update vehicle_roof_datum -> lidar_top tf (calibration)
- Add lidar_front frames and define an estimated tf

File: av_car_description/urdf/mondeo_dca/mondeo_dca_sensors.xacro (robot description, xacro)
@@ -167,6 +167,12 @@
     <origin xyz="0.00939891 0.0238397 0.0606727" rpy="-0.0556599 0.00727062 0.000273152"/>
   </xacro:lidar>
+  <xacro:lidar name="lidar_front_mount" parent="${roof_datum}">
+    <origin xyz="1.777 0 -1.240" rpy="0 0 -3.142"/>
+  </xacro:lidar>
+  <xacro:lidar name="lidar_front" parent="lidar_front_mount">
+    <origin xyz="0 0 0" rpy="0 0 0"/>
+  </xacro:lidar>
   <xacro:lidar name="lidar_top" parent="${roof_datum}">
-    <origin xyz="-0.65855 0 0.26" rpy="0 0 1.5708"/>
+    <origin xyz="-0.65855 0 0.281" rpy="0 0 1.5708"/>
   </xacro:lidar>
   <!-- RADAR -->

Commit message: Compensate `camera_fsp_l` for ground calibration
Generate a new `camera_fsp_l_sensor` to `camera_fsp_l_optical`
  transform using:
  - the updated `vehicle_roof_datum` to `lidar_top` transform
  - the calibration data between `camera_fsp_l_sensor` and `lidar_top`

File: av_car_description/urdf/mondeo_dca/mondeo_dca_sensors.xacro (robot description, xacro)
@@ -15,5 +15,5 @@
   </xacro:camera_mount>
   <xacro:camera_mount name="camera_fsp_l_optical" parent="camera_fsp_l_sensor">
-    <origin xyz="-0.011874 0.049085 0.079928" rpy="0.000929 -0.005284 -0.007228"/>
+    <origin xyz="-0.011877 0.028212 0.077550" rpy="0.000929 -0.005283 -0.007228"/>
   </xacro:camera_mount>
   <xacro:camera_mount name="camera_fsp_r_mount" parent="${roof_datum}">

Commit message: Add estimated lidar left/right tfs

File: av_car_description/urdf/mondeo_dca/mondeo_dca_sensors.xacro (robot description, xacro)
@@ -156,14 +156,14 @@
   <!-- LIDAR -->
   <xacro:lidar name="lidar_left_mount" parent="${roof_datum}">
-    <origin xyz="-0.03015 0.720 -0.22242" rpy="-0.087266 0.087266 0.6562438"/>
+    <origin xyz="-0.03015 0.720 -0.22242" rpy=" 0 0 0"/>
   </xacro:lidar>
   <xacro:lidar name="lidar_left" parent="lidar_left_mount">
-    <origin xyz="0.0288801 -0.0294088 0.110552" rpy="0.0499763 0.0151241 -0.00307838"/>
+    <origin xyz="0 0 0" rpy="0.5443089 0.3911757 2.3500656"/>
   </xacro:lidar>
   <xacro:lidar name="lidar_right_mount" parent="${roof_datum}">
-    <origin xyz="-0.03015 -0.720 -0.22242" rpy="0.087266 0.087266 -0.6562438"/>
+    <origin xyz="-0.03015 -0.720 -0.12242" rpy="0 0 0"/>
   </xacro:lidar>
   <xacro:lidar name="lidar_right" parent="lidar_right_mount">
-    <origin xyz="0.00939891 0.0238397 0.0606727" rpy="-0.0556599 0.00727062 0.000273152"/>
+    <origin xyz="0 0 0" rpy="0.5187668 -0.35907 0.7626228"/>
   </xacro:lidar>
   <xacro:lidar name="lidar_front_mount" parent="${roof_datum}">

Commit message: Update lidar_x_mount -> lidar_x_sensor
- Update based on lidar_top -> lidar_x calibraton
  data

File: av_car_description/urdf/mondeo_dca/mondeo_dca_sensors.xacro (robot description, xacro)
@@ -159,5 +159,5 @@
   </xacro:lidar>
   <xacro:lidar name="lidar_left" parent="lidar_left_mount">
-    <origin xyz="0 0 0" rpy="0.5443089 0.3911757 2.3500656"/>
+    <origin xyz="0.006315 0.052479 0.028250" rpy="0.512480 0.358944 2.339389"/>
   </xacro:lidar>
   <xacro:lidar name="lidar_right_mount" parent="${roof_datum}">
@@ -165,5 +165,5 @@
   </xacro:lidar>
   <xacro:lidar name="lidar_right" parent="lidar_right_mount">
-    <origin xyz="0 0 0" rpy="0.5187668 -0.35907 0.7626228"/>
+    <origin xyz="0.020854 -0.027349 -0.074393" rpy="0.530901 -0.370334 0.800023"/>
   </xacro:lidar>
   <xacro:lidar name="lidar_front_mount" parent="${roof_datum}">
@@ -171,5 +171,5 @@
   </xacro:lidar>
   <xacro:lidar name="lidar_front" parent="lidar_front_mount">
-    <origin xyz="0 0 0" rpy="0 0 0"/>
+    <origin xyz="-0.055467 -0.024169 -0.103460" rpy="0.003800 -0.088963 -0.003051"/>
   </xacro:lidar>
   <xacro:lidar name="lidar_top" parent="${roof_datum}">
